File: PCB (beta)/PCB (beta).sch (EAGLE design)
At the start: 1 part, among them J1 5.5x2.1mm Barrel

Commit message: test
Parts:
- added C1, C12, C2, C3, C7: 0.1uF, SparkFun-Capacitors:0.1UF-0603-25V-(+80/-20%)
- added C10, C17, C23, C8, C9: 10uF, SparkFun-Capacitors:10UF-0603-6.3V-20%
- added C11, C18, C19, C20: 1.0uF, SparkFun-Capacitors:1.0UF-0603-16V-10%
- added C13, C14, C15, C21, C4: 22uF, SparkFun-Capacitors:22UF-0805-6.3V-20%
- added C16: 2.2uF, SparkFun-Capacitors:2.2UF-0603-10V-20%
- added C22: 220PF, SparkFun-Capacitors:270PF-0603-50V-5%
- added C5: 47pF, SparkFun-Capacitors:47PF-0603-50V-5%
- added C6: 100uF, SparkFun-Capacitors:100UF-POLAR-EIA7343-10V-10%(TANT)
- added D1: 5A/20V/550mV, SparkFun-DiscreteSemi:DIODE-SCHOTTKY-B340A
- added F1: 043503.5KRHF, DigiKey:043503.5KRHF
- added PAD1, PAD2, PAD3, PAD4: (no value), wirepad:2,54/1,0
- added R1, R10, R4, R5: 0, SparkFun-Resistors:0OHM-0603-1/10W-5%
- added R2: 18.2k, SparkFun-Resistors:1.8KOHM-0603-1/10W-1%
- added R3: 10k, SparkFun-Resistors:10KOHM-0603-1/10W-1%
- added R6, R7: 100k, SparkFun-Resistors:100KOHM-0603-1/10W-1%
- added R8: 36.5k, SparkFun-Resistors:2.2OHM-0603-1/10W-5%
- added R9: 110k, SparkFun-Resistors:100KOHM-0603-1/10W-1%
- added U$1: TPS63021DSJR, DigiKey:TPS63021DSJR
- added U1: TPS2553DBVT, Texas Instruments_By_element14_Batch_1:TPS2553DBVT
- added U2: TLV62084DSGR, DigiKey:TLV62084DSGR
Connections:
- new net +18V: C18.1, C19.1, C21.1, R7.2, R9.2, U2.VOS
- new net +3V3: C13.1, C14.1, C15.1, C16.1, R6.2, U$1.FB, U$1.VOUT, U$1.VOUT_2
- new net +5V: C6.+, C7.1, C8.1, R3.2, U1.IN, U1.OUT
- new net +VDC_IN_F: C2.1, D1.C, F1.1
- new net +VDC_IN_F_D: D1.A, J1.PWR
- new net AGND: C1.2, C2.2, C3.2, C4.2
- new net EN_1P8V: R10.1, U2.EN
- new net FB_1P8V: R8.2, R9.1, U2.FB
- new net GND: C1.1, C10.2, C11.2, C12.2, C13.2, C14.2, C15.2, C16.2, C18.2, C19.2, C21.2, C5.2, C6.-, C7.2, C8.2, C9.2, J1.GND, R1.1, R2.1, R8.1, U$1.EPAD, U$1.GND, U$1.PS/SYNC, U1.GND, U2.GND, U2.GND_2
- new net GNDINT: PAD3.P, PAD4.P, R1.2
- new net N$1: R5.1, U$1.EN
- new net N$2: R6.1, U$1.PG
- new net N$3: C12.1, U$1.VINA
- new net N$5: R2.2, U1.ILIM
- new net PWRGOOD_1P8V: R7.1, U2.PG
- new net USB3_CONN_EN: R4.1, U1.EN
- new net USB3_CONN_FLT: R3.1, R4.2, U1.~FAULT
- new net V+: C10.1, C11.1, C9.1, U$1.VIN, U$1.VIN_2
- new net VCC: R10.2
- new net VCCINT: C5.1, PAD1.P, PAD2.P
- new net VDD: R5.2
- new net VIN: C3.1, C4.1, F1.2

Commit message: incomplete to page 10
Parts:
- added C24, C25, C26, C27: 0.1uF, SparkFun-Capacitors:0.1UF-0603-25V-(+80/-20%)
- added CF1: NFM18PC104R1E3D, murata-filter:NFM21C
- added D2, D3: 200mA/30V, SparkFun-DiscreteSemi:DIODE-SCHOTTKY-B340A
- added F2: 043503.5KRHF, DigiKey:043503.5KRHF
- added IC1: FT232RQ, ftdichip-3:FT232RQ
- added J2: (no value), SparkFun-Connectors:CONN_03
- added J3: (no value), SparkFun-Connectors:USB_MICRO-B_FEMALE-SMT
- added J4: FEMALE 2x3, SparkFun-Connectors:CONN_03X2FEMALE
- added R11: 100k, SparkFun-Resistors:100KOHM-0603-1/10W-1%
- added R12, R13, R14, R15, R17: 10k, SparkFun-Resistors:10KOHM-0603-1/10W-1%
- added R16: 200k, SparkFun-Resistors:200KOHM-0603-1/10W-1%
- added U$2, U$3, U$5: LFTVS18-1F3_FLIPCHIP, Joule Expansion Board:LFTVS18-1F3_FLIPCHIP
- added U3: LSF0108RKSR, Joule Expansion Board:LSF0108RKSR
Connections:
- new net +VBUS_USBC: F2.2, U$5.P$1
- new net +VBUS_USBC_F: CF1.3, F2.1
- new net +VFTDI_VCC_5P0V: D2.C, D3.C, IC1.VCC
- new net +VUSB_IN_FILT_R: J2.1, R11.1
- new net FTDI_USB_DN: IC1.USBDM
- new net FTDI_USB_DP: IC1.USBDP
- new net FTDI_USB_FILT_DN: J3.D-
- new net FTDI_USB_FILT_DP: J3.D+
- new net N$16: C27.1, R16.1, U3.EN, U3.VREF_B
- new net N$7: J3.ID, R17.2
- new net RST_FT232RQ_N: IC1._RESET, J2.2
- new net UART_2_CTS: U3.A2
- new net UART_2_CTS_LS: IC1._RTS, J4.6, R13.1, U3.B2
- new net UART_2_RTS: U3.A1
- new net UART_2_RTS_LS: IC1._CTS, J4.2, R12.1, U3.B1
- new net UART_2_RXD: U3.A3
- new net UART_2_RXD_LS: IC1.TXD, J4.4, R14.1, U3.B3
- new net UART_2_TXD: U3.A4
- new net UART_2_TXD_LS: IC1.RXD, J4.5, R15.1, U3.B4
- new net VCC/2: C24.1, C25.1, D2.A, IC1.3V3OUT, IC1.VCCIO, J3.VBUS, R11.2
- new net VCCIO: C22.1, C23.1, CF1.1
- net +18V: now also C26.1, U3.VREF_A
- net +3V3: now also R12.2, R13.2, R14.2, R15.2, R16.2
- net +5V: now also D3.A
- net AGND: now also J3.SHIELD, U$5.P$2
- net GND: now also C22.2, C23.2, C24.2, C25.2, C26.2, C27.2, CF1.2@1, IC1.AGND, IC1.GND1, IC1.GND2, IC1.GND3, IC1.TEST, J2.3, J3.GND, J4.1, R17.1, U3.EPAD, U3.GND

Commit message: hi
Parts:
- added C28, C29, C30, C31, C32, C33, C34, C35, C36, C37, C38: 0.1uF, SparkFun-Capacitors:0.1UF-0603-25V-(+80/-20%)
- added P1: 1-2295018-2, 1-2295018-2:1-2295018-2
- added R18, R19, R21: 0, SparkFun-Resistors:0OHM-0603-1/10W-5%
- added R20: 100k, SparkFun-Resistors:100KOHM-0603-1/10W-1%
- added U$10, U$11, U$6, U$7, U$8, U$9: TCE0806S-350-2P-T200, Joule Expansion Board:TCE0806S-350-2P-T200
- added U$12, U$13, U$14, U$15: TCE0806G-900-2P-T200, Joule Expansion Board:TCE0806G-900-2P-T200
- added U$4: (no value), Joule Expansion Board:PI3USB302-AZBEX_ANALOG_SWITCH
Connections:
- new net +VDD_USBC_MUX: C28.1, C29.1, C30.1, R18.1, U$4.VDD_1, U$4.VDD_2, U$4.VDD_3
- new net HDMI_CLK_CONN_DN: U$13.2
- new net HDMI_CLK_CONN_DP: U$13.1
- new net HDMI_CLK_C_DN: C32.2
- new net HDMI_CLK_C_DP: C31.2
- new net HDMI_CLK_DN: C32.1
- new net HDMI_CLK_DP: C31.1
- new net HDMI_DAT0_CONN_DN: U$12.2
- new net HDMI_DAT0_CONN_DP: U$12.1
- new net HDMI_DAT1_CONN_DN: U$14.2
- new net HDMI_DAT1_CONN_DP: U$14.1
- new net HDMI_DAT2_CONN_DN: U$15.2
- new net HDMI_DAT2_CONN_DP: U$15.1
- new net HDMI_OB_CLK_DN: U$13.3
- new net HDMI_OB_CLK_DP: U$13.4
- new net HDMI_OB_DAT0_DN: U$12.3
- new net HDMI_OB_DAT1_DN: U$14.3
- new net HDMI_OB_DAT1_DP: U$14.4
- new net HDMI_OB_DAT2_DN: U$15.3
- new net HDMI_OB_DAT2_DP: U$15.4
- new net HDMI_TX_0_C_DN: C34.2
- new net HDMI_TX_0_C_DP: C33.2
- new net HDMI_TX_0_DN: C34.1
- new net HDMI_TX_0_DP: C33.1
- new net HDMI_TX_1_C_DN: C37.2
- new net HDMI_TX_1_C_DP: C35.2
- new net HDMI_TX_1_DN: C37.1
- new net HDMI_TX_1_DP: C35.1
- new net HDMI_TX_2_C_DN: C38.2
- new net HDMI_TX_2_C_DP: C36.2
- new net HDMI_TX_2_DN: C38.1
- new net HDMI_TX_2_DP: C36.1
- new net TP_USB_TYPC_SBU1_CONN: P1.SBU1
- new net TP_USB_TYPC_SBU2_CONN: P1.SBU2
- new net USB3_0_MUX1_RX_DN: U$4.RX1-, U$7.3
- new net USB3_0_MUX1_RX_DP: U$4.RX1+, U$7.4
- new net USB3_0_MUX1_TX_DN: U$4.TX1-, U$6.3
- new net USB3_0_MUX1_TX_DP: U$4.TX1+, U$6.4
- new net USB3_0_MUX2_RX_DN: U$10.3, U$4.RX2-
- new net USB3_0_MUX2_RX_DP: U$10.4, U$4.RX2+
- new net USB3_0_MUX2_TX_DN: U$4.TX2-, U$8.3
- new net USB3_0_MUX2_TX_DP: U$4.TX2+, U$8.4
- new net USB3_0_RX_DN: U$4.RX-
- new net USB3_0_RX_DP: U$4.RX+
- new net USB3_0_TX_DN: U$4.TX-
- new net USB3_0_TX_DP: U$4.TX+
- new net USB3_1_RX_DN: U$9.4
- new net USB3_1_RX_DP: U$9.3
- new net USB3_1_TX_DN: U$11.4
- new net USB3_1_TX_DP: U$11.3
- new net USBA_USB3_1_RX_DN: U$9.1
- new net USBA_USB3_1_RX_DP: U$9.2
- new net USBA_USB3_1_TX_DN: U$11.1
- new net USBA_USB3_1_TX_DP: U$11.2
- new net USBC_PD: R19.2, U$4.PD
- new net USBC_SEL: R21.1
- new net USBC_SEL_R: R20.2, R21.2, U$4.SEL
- new net USBC_USB2_0_DN: P1.A_D-, P1.B_D-
- new net USBC_USB2_0_DP: P1.A_D+, P1.B_D+
- new net USBC_USB3_0_MUX1_RX_DN: P1.RX1-, U$7.2
- new net USBC_USB3_0_MUX1_RX_DP: P1.RX1+, U$7.1
- new net USBC_USB3_0_MUX1_TX_DN: P1.TX1-, U$6.2
- new net USBC_USB3_0_MUX1_TX_DP: P1.TX1+, U$6.1
- new net USBC_USB3_0_MUX2_RX_DN: P1.RX2-, U$10.2
- new net USBC_USB3_0_MUX2_RX_DP: P1.RX2+, U$10.1
- new net USBC_USB3_0_MUX2_TX_DN: P1.TX2-, U$8.2
- new net USBC_USB3_0_MUX2_TX_DP: P1.TX2+, U$8.1
- new net USB_TYPC_CONN_CC1: P1.CC1
- new net USB_TYPC_CONN_CC2: P1.CC2
- net +3V3: now also R18.2
- net +VBUS_USBC: now also P1.A_VBUS1, P1.A_VBUS2, P1.B_VBUS1, P1.B_VBUS2
- net AGND: now also U$10.5, U$10.6, U$11.5, U$11.6, U$12.5, U$12.6, U$13.5, U$13.6, U$14.5, U$14.6, U$15.5, U$15.6, U$6.5, U$6.6, U$7.5, U$7.6, U$8.5, U$8.6, U$9.5, U$9.6
- net GND: now also C28.2, C29.2, C30.2, P1.A_GND1, P1.A_GND2, P1.B_GND1, P1.B_GND2, R19.1, R20.1, U$4.GND_1, U$4.GND_2, U$4.GND_3, U$4.GND_4
