File: PCB(beta)/PCB(beta).sch (EAGLE design)
At the start: 93 parts, among them IC1 FT232RQ, J1 5.5x2.1mm Barrel, J4 FEMALE 2x3, P1 1-2295018-2, U1 TPS2553DBVT, U2 TLV62084DSGR, U3 LSF0108RKSR

Commit message: 04/03/2017
Parts:
- added C39, C40, C43, C44, C45, C46, C47, C48, C49, C50, C51, C52: 0.1uF, SparkFun-Capacitors:0.1UF-0603-25V-(+80/-20%)
- added C41, C42: 0.22uF, SparkFun-Capacitors:0.22UF-0603-25V-10%
- added D4, D5, D6: 0.5A/40V/420mV, SparkFun-DiscreteSemi:DIODE-SCHOTTKY-PMEG4005EJ
- added J5: (no value), Wurth_Elektronik_Electromechanic_Input-Output_Connectors_rev16b:685119134923
- added R22, R23: 2.7k, SparkFun-Resistors:2.55KOHM-0603-1/10W-1%
- added R24, R29, R30, R39: 200k, SparkFun-Resistors:200KOHM-0603-1/10W-1%
- added R25, R26, R27, R28, R31, R32, R33, R34, R35, R36, R37, R38: 100k, SparkFun-Resistors:100KOHM-0603-1/10W-1%
- added U4, U5, U6, U7, U8: LSF0108RKSR, Joule Expansion Board:LSF0108RKSR
Connections:
- new net CLK_19P2M: U7.A4
- new net CLK_19P2M_LS: U7.B4
- new net CODEC_MCLK: U6.A6
- new net CODEC_MCLK_LS: U6.B6
- new net EN6: C52.1, R39.1, U8.EN, U8.VREF_B
- new net GPIO_22: U7.A1
- new net GPIO_22_LS: U7.B1
- new net HDMI_OB_SCL: J5.SCL, R22.2
- new net HDMI_OB_SDA: J5.SDA, R23.2
- new net I2C_0_SCL: R34.1, U7.A6
- new net I2C_0_SCL_LS: R31.1, U7.B6
- new net I2C_0_SDA: R33.1, U7.A2
- new net I2C_0_SDA_LS: R32.1, U7.B2
- new net I2S_1_CLK: U6.A7
- new net I2S_1_CLK_LS: U6.B7
- new net I2S_1_FS: U6.A5
- new net I2S_1_FS_LS: U6.B5
- new net I2S_1_RXD: U6.A4
- new net I2S_1_RXD_LS: U6.B4
- new net I2S_1_TXD: U6.A3
- new net I2S_1_TXD_LS: U6.B3
- new net ISH_GPIO_0: U8.A4
- new net ISH_GPIO_0_LS: U8.B4
- new net ISH_GPIO_1: U8.A3
- new net ISH_GPIO_1_LS: U8.B3
- new net ISH_GPIO_2: U4.A6
- new net ISH_GPIO_2_LS: U4.B6
- new net ISH_GPIO_3: U4.A5
- new net ISH_GPIO_3_LS: U4.B5
- new net ISH_GPIO_4_LS: U8.B2
- new net ISH_GPIO_5: U4.A4
- new net ISH_GPIO_5_LS: U4.B4
- new net ISH_GPIO_6: U8.A1
- new net ISH_GPIO_6_LS: U8.B1
- new net ISH_I2C_0_SCL: R25.1, U5.A4
- new net ISH_I2C_0_SCL_LS: R27.1, U5.B4
- new net ISH_I2C_0_SDA: R26.1, U5.A3
- new net ISH_I2C_0_SDA_LS: R28.1, U5.B3
- new net ISH_I2C_1_SCL: R36.1, U8.A6
- new net ISH_I2C_1_SCL_LS: R37.1, U8.B6
- new net ISH_I2C_1_SDA: R35.1, U8.A5
- new net ISH_I2C_1_SDA_LS: R38.1, U8.B5
- new net ISK_GPIO_4: U8.A2
- new net N$10: D5.C, R23.1
- new net N$11: C48.1, R30.1, U6.EN, U6.VREF_B
- new net N$12: C46.1, R29.1, U5.EN, U5.VREF_B
- new net N$13: C43.1, R24.1, U4.EN, U4.VREF_B
- new net N$4: J5.DDC/CECGROUND
- new net N$6: C40.1, C41.1, C42.1, D6.C, J5.+5VPOWER
- new net N$9: D4.C, R22.1
- new net PMIC_PWRGOOD: U6.A8
- new net PMIC_PWRGOOD_LS: U6.B8
- new net PMIC_RESET_N: U4.A1
- new net PMIC_RESET_N_LS: U4.B1
- new net PWM_0: U4.A3
- new net PWM_0_LS: U4.B3
- new net PWM_1: U4.A2
- new net PWM_1_LS: U4.B2
- new net PWM_2: U5.A2
- new net PWM_2_LS: U5.B2
- new net PWM_3: U5.A1
- new net PWM_3_LS: U5.B1
- new net SPI_1_CLK: U6.A1
- new net SPI_1_CLK_LS: U6.B1
- new net SPI_1_FS0: U7.A8
- new net SPI_1_FS0_LS: U7.B8
- new net SPI_1_FS2: U5.A5
- new net SPI_1_FS2_LS: U5.B5
- new net SPI_1_MISO: U7.A5
- new net SPI_1_MISO_LS: U7.B5
- new net SPI_1_MOSI: U6.A2
- new net SPI_1_MOSI_LS: U6.B2
- new net TP_HDMI_CEC: J5.CEC
- new net UART_0_TXD: U7.A3
- new net UART_0_TXD_LS: U7.B3
- new net UART_1_RXD: U4.A8
- new net UART_1_RXD_LS: U4.B8
- new net UART_1_TXD: U4.A7
- new net UART_1_TXD_LS: U4.B7
- net +18V: now also C44.1, C45.1, C47.1, C49.1, C51.1, R25.2, R26.2, R33.2, R34.2, R35.2, R36.2, U4.VREF_A, U5.VREF_A, U6.VREF_A, U7.VREF_A, U8.VREF_A
- net +3V3: now also C50.1, R24.2, R27.2, R28.2, R29.2, R30.2, R31.2, R32.2, R37.2, R38.2, R39.2, U7.EN, U7.VREF_B
- net +5V: now also C39.1, D4.A, D5.A, D6.A
- net GND: now also C39.2, C40.2, C41.2, C42.2, C43.2, C44.2, C45.2, C46.2, C47.2, C48.2, C49.2, C50.2, C51.2, C52.2, J5.TMDSCLOCKSHIELD, J5.TMDSDATA0SHIELD, J5.TMDSDATA1SHIELD, J5.TMDSDATA2SHIELD, U4.EPAD, U4.GND, U5.EPAD, U5.GND, U6.EPAD, U6.GND, U7.EPAD, U7.GND, U8.EPAD, U8.GND
- net HDMI_CLK_CONN_DN: now also J5.TMDSCLOCK-
- net HDMI_CLK_CONN_DP: now also J5.TMDSCLOCK+
- net HDMI_DAT0_CONN_DN: now also J5.TMDSDATA0-
- net HDMI_DAT0_CONN_DP: now also J5.TMDSDATA0+
- net HDMI_DAT1_CONN_DN: now also J5.TMDSDATA1-
- net HDMI_DAT1_CONN_DP: now also J5.TMDSDATA1+
- net HDMI_DAT2_CONN_DN: now also J5.TMDSDATA2-
- net HDMI_DAT2_CONN_DP: now also J5.TMDSDATA2+

Commit message: 04/03/2017
Parts:
- added C53, C54, C55, C56: 0.1uF, SparkFun-Capacitors:0.1UF-0603-25V-(+80/-20%)
- added D10, D7, D8, D9: GREEN, SparkFun-LED:LED-GREEN0603
- added J6: SSM-120-S-DV, Joule Expansion Board:SSM-120-S-DV
- added Q1, Q2: (no value), SparkFun-DiscreteSemi:TRANS_NPN_DUAL-MBT3904DW1T1
- added R40, R41, R42, R43: 1.1k, SparkFun-Resistors:1.5KOHM-0603-1/10W-1%
- added R44, R45, R46, R47: 560, SparkFun-Resistors:510OHM-2010-1/2W-5%
Connections:
- new net ISH_GPIO0_COL: D7.A, R44.1
- new net ISH_GPIO0_COL_D: D7.C, Q1Q1.C
- new net ISH_GPIO1_COL: D8.A, R45.1
- new net ISH_GPIO1_COL_D: D8.C, Q1Q2.C
- new net ISH_GPIO_0_R: Q1Q1.B, R40.2
- new net ISH_GPIO_1_R: Q1Q2.B, R41.2
- net +5V: now also R44.2, R45.2, R46.2, R47.2
- net CLK_19P2M_LS: now also J6.5
- net CODEC_MCLK_LS: now also J6.20
- net GND: now also C53.2, C54.2, C55.2, C56.2, J6.36, J6.37, J6.38, J6.39, Q1Q1.E, Q1Q2.E
- net GPIO_22_LS: now also J6.1
- net I2C_0_SCL_LS: now also J6.13
- net I2C_0_SDA_LS: now also J6.11
- net I2S_1_CLK_LS: now also J6.18
- net I2S_1_FS_LS: now also J6.16
- net I2S_1_RXD_LS: now also J6.12
- net I2S_1_TXD_LS: now also J6.14
- net ISH_GPIO_0: now also R40.1
- net ISH_GPIO_0_LS: now also J6.35
- net ISH_GPIO_1: now also R41.1
- net ISH_GPIO_1_LS: now also J6.33
- net ISH_GPIO_2_LS: now also J6.31
- net ISH_GPIO_3_LS: now also J6.29
- net ISH_GPIO_4_LS: now also J6.27
- net ISH_GPIO_5_LS: now also J6.25
- net ISH_GPIO_6_LS: now also J6.23
- net ISH_I2C_0_SCL_LS: now also J6.17
- net ISH_I2C_0_SDA_LS: now also J6.15
- net ISH_I2C_1_SCL_LS: now also J6.21
- net ISH_I2C_1_SDA_LS: now also J6.19
- net PMIC_PWRGOOD_LS: now also J6.9
- net PMIC_RESET_N_LS: now also J6.3
- net PWM_0_LS: now also J6.26
- net PWM_1_LS: now also J6.28
- net PWM_2_LS: now also J6.30
- net PWM_3_LS: now also J6.32
- net SPI_1_CLK_LS: now also J6.10
- net SPI_1_FS0_LS: now also J6.6
- net SPI_1_FS2_LS: now also J6.8
- net SPI_1_MISO_LS: now also J6.2
- net SPI_1_MOSI_LS: now also J6.4
- net UART_0_TXD_LS: now also J6.7
- net UART_1_RXD_LS: now also J6.24
- net UART_1_TXD_LS: now also J6.22
- net VCC: now also C55.1, C56.1, J6.34
- net VDD: now also C53.1, C54.1, J6.40

Commit message: 04/03/2017
Parts:
- added C57, C58, C59, C60, C61, C62, C63, C64, C65, C66, C67, C68, C69, C70, C71: 0.1uF, SparkFun-Capacitors:0.1UF-0603-25V-(+80/-20%)
- added J7: SSM-120-S-DV, Joule Expansion Board:SSM-120-S-DV
- added R48, R49, R50, R51, R52, R53, R58, R59, R60: 100k, SparkFun-Resistors:100KOHM-0603-1/10W-1%
- added R54, R55, R56, R57: 200k, SparkFun-Resistors:200KOHM-0603-1/10W-1%
- added R61: 100, SparkFun-Resistors:100OHM-0603-1/4W-5%
- added R62, R63: 3.3k, SparkFun-Resistors:3.3KOHM-0603-1/10W-1%
- added R64, R65, R66, R67: 10k, SparkFun-Resistors:10KOHM-0603-1/10W-1%
- added R68, R69, R70, R71, R72, R73, R74: 0, SparkFun-Resistors:0OHM-0603-1/10W-5%
- added S1, S2, S3: (no value), SparkFun-Switches:MOMENTARY-SWITCH-SPST-2-SMD-4.6X2.8MM
- added U$16: TSM-102-01-L-DV-TR, Joule Expansion Board:TSM-102-01-L-DV-TR
- added U$17: M24M02-DRMN6TP, Joule Expansion Board:M24M02-DRMN6TP
- added U10, U11, U12, U9: LSF0108RKSR, Joule Expansion Board:LSF0108RKSR
Connections:
- new net AVS_M_CLK_A1: U10.A1
- new net AVS_M_CLK_A1_LS: J7.26, U10.B1
- new net AVS_M_CLK_B1: U10.A6
- new net AVS_M_CLK_B1_LS: J7.24, U10.B6
- new net AVS_M_DATA_1: U10.A7
- new net AVS_M_DATA_1_LS: J7.22, U10.B7
- new net BLDRW_0_PWM: U10.A3
- new net BLDRW_0_PWM_LS: J7.17, U10.B3
- new net BTN_N: R60.1, S2.3, S2.4
- new net DISPLAY_0_BIAS_EN: U10.A2
- new net DISPLAY_0_BIAS_EN_LS: J7.13, U10.B2
- new net DISPLAY_0_BKLT_EN: U10.A4
- new net DISPLAY_0_BKLT_EN_LS: J7.15, U10.B4
- new net DISPLAY_0_RST_N: U10.A8
- new net DISPLAY_0_RST_N_LS: J7.11, U10.B8
- new net EEPROM_E2: R66.1, R67.2, U$17.E2
- new net EEPROM_VCC: R69.1, U$17.VCC
- new net EEPROM_WC_N: R64.1, R65.2, U$17./WC
- new net FLASH_RST_N: U11.A2
- new net FLASH_RST_N_LS: J7.18, U11.B2
- new net FLASH_TORCH: U11.A3
- new net FLASH_TORCH_LS: J7.16, U11.B3
- new net FLASH_TRIGGER: U11.A1
- new net FLASH_TRIGGER_LS: J7.20, U11.B1
- new net I2C_0_SDA_EE_R: R68.1, U$17.SDA
- new net I2C_1_SCL: R48.1, U9.A8
- new net I2C_1_SCL_LS: J7.33
- new net I2C_1_SDA: R58.1, U12.A1
- new net I2C_1_SDA_LS: J7.31, R59.1, U12.B1
- new net I2C_2_SCL: R49.1, U9.A6
- new net I2C_2_SCL_LS: J7.37, R51.1, U9.B6
- new net I2C_2_SDA: R50.1, U9.A7
- new net I2C_2_SDA_LS: J7.35, R52.1, R53.1, U9.B7, U9.B8
- new net ISH_GPIO2_COL: D9.A, R46.1
- new net ISH_GPIO2_COL_D: D9.C, Q2Q1.C
- new net ISH_GPIO3_COL: D10.A, R47.1
- new net ISH_GPIO3_COL_D: D10.C, Q2Q2.C
- new net ISH_GPIO_2_R: Q2Q1.B, R42.2
- new net ISH_GPIO_3_R: Q2Q2.B, R43.2
- new net ISH_UART_0_CTS: U9.A2
- new net ISH_UART_0_CTS_LS: J7.40, U9.B2
- new net ISH_UART_0_RTS: U9.A3
- new net ISH_UART_0_RTS_LS: J7.38, U9.B3
- new net ISH_UART_0_RXD: U9.A4
- new net ISH_UART_0_RXD_LS: J7.36, U9.B4
- new net ISH_UART_0_TXD: U9.A5
- new net ISH_UART_0_TXD_LS: J7.34, U9.B5
- new net N$14: C60.1, R55.1, U10.EN, U10.VREF_B
- new net N$17: C64.1, R57.1, U12.EN, U12.VREF_B
- new net N$18: R70.2, U$17.SCL
- new net N$19: C58.1, R54.1, U9.EN, U9.VREF_B
- new net N$8: C62.1, R56.1, U11.EN, U11.VREF_B
- new net PMIC_PWRBTN_N: S1.3, S1.4
- new net PMIC_SLPCLK_1: U9.A1
- new net PMIC_SLPCLK_1_LS: U9.B1
- new net PMIC_SPLCLK_1_LS: J7.39
- new net SPI_0_CLK: U12.A8
- new net SPI_0_CLK_LS: J7.25, U12.B8
- new net SPI_0_FS0: U11.A4
- new net SPI_0_FS0_LS: J7.19, U11.B4
- new net SPI_0_FS1: U10.A5
- new net SPI_0_FS1_LS: J7.21, U10.B5
- new net SPI_0_FS2: U12.A5
- new net SPI_0_FS2_LS: J7.23, U12.B5
- new net SPI_0_MISO: U12.A3
- new net SPI_0_MISO_LS: J7.29, U12.B3
- new net SPI_0_MOSI: U12.A7
- new net SPI_0_MOSI_LS: J7.27, U12.B7
- new net SPI_1_FS2_PD: R62.2, U$16.P$4
- new net UART_0_CTS: U12.A2
- new net UART_0_CTS_LS: J7.32, U12.B2
- new net UART_0_RTS: U12.A6
- new net UART_0_RTS_LS: J7.30, U12.B6
- new net UART_0_RXD: U12.A4
- new net UART_0_RXD_LS: J7.28, U12.B4
- new net UART_1_TXD_PD: R63.2, U$16.P$2
- new net UART_2_TXD_PU: R61.1, S3.3, S3.4
- net +18V: now also C57.1, C59.1, C61.1, C63.1, C65.1, C66.1, J7.12, R48.2, R49.2, R50.2, R58.2, U10.VREF_A, U11.VREF_A, U12.VREF_A, U9.VREF_A
- net +3V3: now also C67.1, C68.1, J7.6, J7.8, R51.2, R52.2, R53.2, R54.2, R55.2, R56.2, R57.2, R59.2
- net +5V: now also C69.1, C70.1, J7.2, J7.4
- net AGND: now also R71.2, R72.2, R73.2, R74.2
- net GND: now also C57.2, C58.2, C59.2, C60.2, C61.2, C62.2, C63.2, C64.2, C65.2, C66.2, C67.2, C68.2, C69.2, C70.2, C71.2, J7.1, J7.14, J7.3, J7.5, J7.7, J7.9, Q2Q1.E, Q2Q2.E, R65.1, R67.1, R71.1, R72.1, R73.1, R74.1, S1.1, S1.2, S2.1, S2.2, U$17.VSS, U10.EPAD, U10.GND, U11.EPAD, U11.GND, U12.EPAD, U12.GND, U9.EPAD, U9.GND
- net I2C_0_SCL: now also R70.1
- net I2C_0_SDA: now also R68.2
- net ISH_GPIO_2: now also R42.1
- net ISH_GPIO_3: now also R43.1
- net SPI_1_FS2: now also U$16.P$3
- net UART_1_TXD: now also U$16.P$1
- net UART_2_TXD: now also S3.1, S3.2
- net VCC: now also C71.1, R60.2, R61.2, R64.2, R66.2, R69.2

Commit message: final stages
Parts:
- added C72, C76, C89: 10uF, SparkFun-Capacitors:10UF-0603-6.3V-20%
- added C73, C74: 2.2uF, SparkFun-Capacitors:2.2UF-0603-10V-20%
- added C75: 100uF, SparkFun-Capacitors:100UF-POLAR-10X10.5-63V-20%
- added C77: 100pF, SparkFun-Capacitors:100PF-0603-50V-5%
- added C78, C79, C80: 22uF, SparkFun-Capacitors:22UF-0805-6.3V-20%
- added C81, C86, C87, C88, C90: 0.1uF, SparkFun-Capacitors:0.1UF-0603-25V-(+80/-20%)
- added C82: 47pF, SparkFun-Capacitors:47PF-0603-50V-5%
- added C83: 1.0uF, SparkFun-Capacitors:1.0UF-0603-16V-10%
- added C84, C85: 220pF, SparkFun-Capacitors:180PF-0603-50V-5%
- added FB1, FB2, FB3, FB4, FB5: 120Ω/1.3A, SparkFun-Coils:FERRITE_BEAD-0603
- added H1, H2, H3, H4: MOUNT-PAD-ROUND4.1, holes:MOUNT-PAD-ROUND4.1
- added J8: (no value), SparkFun-Connectors:CONN_03SMD
- added K1: 692122030100, Wuerth_Elektronik_eiCan_Communication_Connectors_STENCIL:692122030100
- added R75, R76, R80, R85, R86, R87, R88, R89, R91: 0, SparkFun-Resistors:0OHM-0603-1/10W-5%
- added R77, R93, R96: 10k, SparkFun-Resistors:10KOHM-0603-1/10W-1%
- added R78, R84, R92: 1k, SparkFun-Resistors:1KOHM-0603-1/10W-1%
- added R79: 1.5k, SparkFun-Resistors:1.5KOHM-0603-1/10W-1%
- added R81, R82, R90, R94: 100k, SparkFun-Resistors:100KOHM-0603-1/10W-1%
- added R83: 200k, SparkFun-Resistors:200KOHM-0603-1/10W-1%
- added R95: 1.1k, SparkFun-Resistors:1KOHM-0603-1/10W-1%
- added U$18: FPF3042UCX, Joule Expansion Board:FPF3042UCX
- added U$19, U$20: FPF2495UCX, Joule Expansion Board:FPF2495UCX
- added U$21: FAN48623UC50X_SWITCHING_REGULATOR, Joule Expansion Board:FAN48623UC50X_SWITCHING_REGULATOR
- added U$22, U$23: SPM4012T-1R0M, Joule Expansion Board:SPM4012T-1R0M
- added U$24, U$25, U$26: ECMF02-2BF3, Joule Expansion Board:ECMF02-2BF3
- added U$27: IP4856CX25, Joule Expansion Board:IP4856CX25
- added U$28: SSM3K56CTL3FCT-ND_NCHAN_MOSFET, Joule Expansion Board:SSM3K56CTL3FCT-ND_NCHAN_MOSFET
- added U$29, U$31, U$32, U$33, U$34, U$35, U$36, U$37, U$38, U$39, U$40, U$41, U$42, U$43, U$44: (no value), Joule Expansion Board:LXES15AAA1-100_ESD_SUPPRESSOR
- added U$30: BK-916-TR_12MM_COINCELL, Joule Expansion Board:BK-916-TR_12MM_COINCELL
- added U$45, U$46, U$47, U$48: 92320A282_1/8_SPACER, Joule Expansion Board:92320A282_1/8_SPACER
- U2: device DigiKey:TLV62084DSGR -> Joule Expansion Board:TLV62084DSGR
Connections:
- net N$1 renamed EN_3P3V
- net N$10 renamed HDMI_OB_SDA_D
- net N$18 renamed I2C_0_SCL_EE_R
- net N$2 renamed PWRGOOD_3P3V
- net N$3 renamed +V3P3V_VINA
- net N$6 renamed +V5P0V_D
- net N$7 renamed FTDI_USB_ID
- net N$9 renamed HDMI_OB_SCL_D
- removed net +18V: C18.1, C19.1, C21.1, C26.1, C44.1, C45.1, C47.1, C49.1, C51.1, C57.1, C59.1, C61.1, C63.1, C65.1, C66.1, J7.12, R25.2, R26.2, R33.2, R34.2, R35.2, R36.2, R48.2, R49.2, R50.2, R58.2, R7.2, R9.2, U10.VREF_A, U11.VREF_A, U12.VREF_A, U2.VOS, U3.VREF_A, U4.VREF_A, U5.VREF_A, U6.VREF_A, U7.VREF_A, U8.VREF_A, U9.VREF_A
- removed net VIN: C3.1, C4.1, F1.2
- new net +1.8V: C18.1, C19.1, C21.1, C26.1, C44.1, C45.1, C47.1, C49.1, C51.1, C57.1, C59.1, C61.1, C63.1, C65.1, C66.1, FB5.1, J7.12, R25.2, R26.2, R33.2, R34.2, R35.2, R36.2, R48.2, R49.2, R50.2, R58.2, R7.2, R9.2, R92.2, R93.2, U$23.1, U$37.P$1, U10.VREF_A, U11.VREF_A, U12.VREF_A, U2.VOS, U3.VREF_A, U4.VREF_A, U5.VREF_A, U6.VREF_A, U7.VREF_A, U8.VREF_A, U9.VREF_A
- new net +V1P8V_MICROSD: C87.1, FB5.2, U$27.VCCA
- new net +V1P8V_SW: U$23.2, U2.SW
- new net +V3P3V_FT23RQ: C24.1, C25.1, IC1.3V3OUT, IC1.VCCIO
- new net +V3P3V_MICROSD: C88.1, C89.1, FB4.2, U$27.VSD_REF, U$27.VSUPPLY, U$34.P$1
- new net +V3P3V_SW_L1: U$1.L1, U$1.L1_2, U$22.2
- new net +V3P3V_SW_L2: U$1.L2, U$1.L2_2, U$22.1
- new net +V5P0V_USBA: C81.1, K1.VBUS
- new net +VBUS: C75.+, U$18.VBUS_1, U$18.VBUS_2, U$18.VBUS_3, U$20.VOUT1, U$20.VOUT2
- new net +VDC_IN: C3.1, C4.1, C72.1, F1.2, U$18.VIN_3
- new net +VDD1: C55.1, C56.1, C71.1, J6.34, R10.2, R64.2, R66.2, R69.2, U$35.P$1
- new net +VDD3: C53.1, C54.1, J6.40, R81.2, U$36.P$1
- new net +VIN_CHRG: U$18.VOUT_1, U$18.VOUT_2, U$18.VOUT_3, U$18.VOUT_4
- new net +VLDO_SDCARD: C83.1, U$27.VLDO
- new net +VSYS: C17.1, C20.1, C76.1, C77.1, R86.2, R87.2, U$21.VIN, U$21.VIN1, U2.1
- new net +VUSB_IN: FB3.2, J3.VBUS, U$33.P$1
- new net +VUSB_IN_FILT: C86.1, D2.A, FB3.1, R11.2
- new net BOOST_DCDC_BYP_N: R84.1, R85.2, U$21.BYP_N
- new net CHS_GND: C1.2, C2.2, J3.SHIELD, R71.2, R72.2, R73.2, R74.2, U$10.5, U$10.6, U$11.5, U$11.6, U$12.5, U$12.6, U$13.5, U$13.6, U$14.5, U$14.6, U$15.5, U$15.6, U$24.GND, U$25.GND, U$31.P$2, U$32.P$2, U$33.P$2, U$34.P$2, U$5.P$2, U$6.5, U$6.6, U$7.5, U$7.6, U$8.5, U$8.6, U$9.5, U$9.6
- new net DF_IN: R75.2, U$18.DF_IN
- new net EN_5P0V: R81.1, R83.2, U$21.EN
- new net FAN_CTRL: J8.2, R96.1
- new net HPD_SRC: R92.1, U$28.D
- new net HPD_SRC_N: R93.1, R94.2, U$28.G
- new net N$1: R95.2, U$29.P$1, U$30.+
- new net OTG_EN: R80.1
- new net OTG_EN_R: R80.2, U$20.ON
- new net OTG_I_ADJ: R78.2, U$20.ISET
- new net OTG_OCFLAG_TP: U$20.OCFLAGB
- new net PWRGOOD_5P0V: R82.1, U$21.PG
- new net SCARD_CD_N_CONN: R89.2, U$27.CD
- new net SDCARD_CD_N: R89.1
- new net SDCARD_CLK: U$27.CLK_IN
- new net SDCARD_CLK_CONN: C82.1, R91.2
- new net SDCARD_CLK_CONN_R: R91.1, U$27.CLK_SD
- new net SDCARD_CMD: U$27.CMD_H
- new net SDCARD_CMD_CONN: U$27.CMD_SD
- new net SDCARD_D0: U$27.DATA0_H
- new net SDCARD_D0_CONN: U$27.DATA0_SD
- new net SDCARD_D1: U$27.DATA1_H
- new net SDCARD_D1_CONN: U$27.DATA1_SD
- new net SDCARD_D2: U$27.DATA2_H
- new net SDCARD_D2_CONN: U$27.DATA2_SD
- new net SDCARD_D3: U$27.DATA3_H
- new net SDCARD_D3_CONN: U$27.DATA3_SD
- new net SDCARD_LVL_CLK_FB: U$27.CLK_FB
- new net SDCARD_LVL_CMD_DIR: U$27.DIR_CMD
- new net SDCARD_LVL_DAT_DIR: U$27.DIR_0, U$27.DIR_1_3
- new net SDCARD_LVL_SEL: U$27.SEL
- new net SDCARD_PWR_DOWN_N: R88.1, R90.2
- new net SDCARD_PWR_DOWN_N_R: R88.2, U$27.ENABLE
- new net USB2_0_DN: U$24.OUT2
- new net USB2_0_DP: U$24.OUT1
- new net USB2_1_DN: U$25.IN1
- new net USB2_1_DP: U$25.IN2
- new net USBA_USB2_1_DN: K1.D-, U$25.OUT1
- new net USBA_USB2_1_DP: K1.D+, U$25.OUT2
- new net USB_TYPC_CC1: C85.1, FB2.2
- new net USB_TYPC_CC2: C84.1, FB1.2
- new net VCONN_DCDC_EN: U$19.ON
- new net VCONN_I_ADJ: R79.2, U$19.ISET
- new net VCONN_OCFLAG_TP: U$19.OCFLAGB
- new net VIN_EN: R77.2, U$18.EN
- new net VIN_SEL: R76.2, U$18.VIN_SEL
- new net VSEL_5P0V: R86.1, R87.1, U$21.VSEL
- net +3V3: now also FB4.1, R96.2, U$38.P$1
- net +5V: now also C73.1, C74.1, C78.1, C79.1, C80.1, C90.1, J8.1, R82.2, U$19.VIN1, U$19.VIN2, U$20.VIN1, U$20.VIN2, U$21.VOUT, U$21.VOUT1, U$39.P$1
- net +VDC_IN_F: now also U$2.P$1
- net AGND: now also U$2.P$2, U$26.GND, U$3.P$2; no longer C1.2, C2.2, C3.2, C4.2, J3.SHIELD, R71.2, R72.2, R73.2, R74.2, U$10.5, U$10.6, U$11.5, U$11.6, U$12.5, U$12.6, U$13.5, U$13.6, U$14.5, U$14.6, U$15.5, U$15.6, U$5.P$2, U$6.5, U$6.6, U$7.5, U$7.6, U$8.5, U$8.6, U$9.5, U$9.6
- net BTN_N: now also U$41.P$1
- net FTDI_USB_DN: now also U$26.OUT1
- net FTDI_USB_DP: now also U$26.OUT2
- net FTDI_USB_FILT_DN: now also U$26.IN1
- net FTDI_USB_FILT_DP: now also U$26.IN2
- net GND: now also C17.2, C20.2, C3.2, C4.2, C72.2, C73.2, C74.2, C75.-, C76.2, C77.2, C78.2, C79.2, C80.2, C81.2, C82.2, C83.2, C84.2, C85.2, C86.2, C87.2, C88.2, C89.2, C90.2, H1.MOUNT, H2.MOUNT, H3.MOUNT, H4.MOUNT, J8.3, K1.GND, K1.GND_DRAIN, R62.1, R63.1, R75.1, R76.1, R77.1, R78.1, R79.1, R83.1, R85.1, R90.1, R94.1, U$18.GND_1, U$18.GND_2, U$19.GND1, U$19.GND2, U$20.GND1, U$20.GND2, U$21.AGND, U$21.NC_PGND, U$21.NC_PGND1, U$21.PGND, U$21.PGND1, U$21.PGND2, U$27.GND, U$28.S, U$29.P$2, U$3.P$1, U$30.-, U$35.P$2, U$36.P$2, U$37.P$2, U$38.P$2, U$39.P$2, U$40.P$2, U$41.P$2, U$42.P$2, U$43.P$2, U$44.P$2, U$45.1, U$46.1, U$47.1, U$48.1
- net PMIC_PWRBTN_N: now also U$42.P$1
- net SPI_1_FS2: now also U$44.P$1
- net UART_1_TXD: now also U$43.P$1
- net UART_2_TXD: now also U$40.P$1
- net USBA_USB3_1_RX_DN: now also K1.STDA_SSRX-, K1.STDA_SSTX-
- net USBA_USB3_1_RX_DP: now also K1.STDA_SSRX+, K1.STDA_SSTX+
- net USBC_USB2_0_DN: now also U$24.IN2
- net USBC_USB2_0_DP: now also U$24.IN1
- net USB_TYPC_CONN_CC1: now also FB2.1, U$32.P$1
- net USB_TYPC_CONN_CC2: now also FB1.1, U$31.P$1
- net V+: now also R84.2, R95.1
- net VCC: no longer C55.1, C56.1, C71.1, J6.34, R10.2, R64.2, R66.2, R69.2
- net VCC/2: now also U$19.VOUT1, U$19.VOUT2; no longer C24.1, C25.1, D2.A, IC1.3V3OUT, IC1.VCCIO, J3.VBUS, R11.2
- net VDD: no longer C53.1, C54.1, J6.40
Other:
- moved on the sheet: C22, C23, CF1, J1

Commit message: final stages
Parts:
- added C91: 0.1uF, SparkFun-Capacitors:0.1UF-0603-25V-(+80/-20%)
- added C92, C93, C94, C99: 10uF, SparkFun-Capacitors:10UF-0603-6.3V-20%
- added C95: 47nF, SparkFun-Capacitors:47NF-0603-25V-5%
- added C96: 4.7uF, SparkFun-Capacitors:4.7UF0603
- added C97, C98: 22uF, SparkFun-Capacitors:22UF-0805-6.3V-20%
- added D11: (no value), SparkFun-LED:LED0603
- added J9: DM3AT-SF-PEJM5, connector:DM3AT-SF-PEJM5
- added R100: 10k, SparkFun-Resistors:10KOHM-0603-1/10W-1%
- added R101, R102, R103, R104, R106, R97: 100k, SparkFun-Resistors:100KOHM-0603-1/10W-1%
- added R105: 100, SparkFun-Resistors:100OHM-0603-1/4W-5%
- added R107: 120k, SparkFun-Resistors:100KOHM-0603-1/10W-1%
- added R108, R98: 0, SparkFun-Resistors:0OHM-0603-1/10W-5%
- added R99: 510, SparkFun-Resistors:510OHM-2010-1/2W-5%
- added U$49: ASPIAIG-S8050, Joule Expansion Board:ASPIAIG-S8050
- added U$50: (no value), Joule Expansion Board:LXES15AAA1-100_ESD_SUPPRESSOR
- added U$51: BQ25892RTWT, Joule Expansion Board:BQ25892RTWT
- added U$52: SSM3K56CTL3FCT-ND_NCHAN_MOSFET, Joule Expansion Board:SSM3K56CTL3FCT-ND_NCHAN_MOSFET
- added U$53: SPM4012T-1R0M, Joule Expansion Board:SPM4012T-1R0M
- R92: value 1k -> 1.1k
Connections:
- net GNDINT renamed BATT_GND
- net VCC/2 renamed +V5P0V_CONN
- removed net AGND: U$2.P$2, U$26.GND, U$3.P$2
- removed net SCARD_CD_N_CONN: R89.2, U$27.CD
- removed net VCC: R60.2, R61.2
- removed net VCCINT: C5.1, PAD1.P, PAD2.P
- removed net VCCIO: C22.1, C23.1, CF1.1
- removed net VDD: R5.2
- new net +V5P0V_SW: U$21.SW, U$21.SW1, U$49.2
- new net +VBATTERY: C5.1, PAD1.P, PAD2.P, U$50.P$1
- new net +VBOOST: C95.2, U$51.BTST
- new net +VREGN: C96.1, R100.2, R101.2, R106.2, R99.2, U$51.REGN
- new net +VRTC: R95.1
- new net +V_CHRG_LX: C95.1, U$51.SW_1, U$51.SW_2, U$53.2
- new net CHRG_EN_N: R104.2, U$52.G
- new net CHRG_EN_N_R: R103.1, U$51.CE*, U$52.D
- new net CHRG_ILIM: R105.2, U$51.ILIM
- new net CHRG_INT_N: U$51.INT
- new net CHRG_LED_A: D11.A, R99.1
- new net CHRG_OTG: R102.1, U$51.OTG
- new net CHRG_PG_N: D11.C, R100.1, U$51.PG*
- new net CHRG_PMID: C94.1, U$51.PMID
- new net CHRG_PSEL: R97.1, R98.2, U$51.PSEL
- new net CHRG_QON: R108.1, U$51.QON*
- new net CHRG_STAT: R101.1, U$51.STAT
- new net CHRG_TS: R106.1, R107.2, U$51.TS
- new net SDCARD_CD_N_CONN: J9.A, R89.2, U$27.CD
- net +5V: no longer C6.+, C7.1, U1.OUT
- net +V3P3V_MICROSD: now also J9.VCC
- net +V5P0V_USBA: now also C6.+, C7.1, U1.OUT
- net +VBUS: now also C22.1, C23.1, CF1.1
- net +VDD1: now also R60.2, R61.2
- net +VDD3: now also R5.2
- net +VIN_CHRG: now also C91.1, C92.1, C93.1, U$51.VBUS
- net +VSYS: now also C10.1, C11.1, C9.1, C97.1, C98.1, R102.2, R103.2, R84.2, R97.2, U$1.VIN, U$1.VIN_2, U$49.1, U$51.SYS_1, U$51.SYS_2, U$53.1
- net CHS_GND: now also U$2.P$2, U$26.GND, U$3.P$2
- net GND: now also C91.2, C92.2, C93.2, C94.2, C96.2, C97.2, C98.2, C99.2, J9.B, J9.GND, R104.1, R105.1, R107.1, R98.1, U$50.P$2, U$51.EP_GND, U$51.PGND_1, U$52.S
- net I2C_0_SCL: now also U$51.SCL
- net I2C_0_SDA: now also U$51.SDA
- net PMIC_PWRBTN_N: now also R108.2
- net SDCARD_CLK_CONN: now also J9.CLK
- net SDCARD_CMD_CONN: now also J9.CMD/MOSI
- net SDCARD_D0_CONN: now also J9.DATA0/MISO
- net SDCARD_D1_CONN: now also J9.DATA1/RSV
- net SDCARD_D2_CONN: now also J9.DATA2/NC
- net SDCARD_D3_CONN: now also J9.DATA3-CD/CS_N
- net V+: now also C99.1, U$51.BAT_1, U$51.BAT_2; no longer C10.1, C11.1, C9.1, R84.2, R95.1, U$1.VIN, U$1.VIN_2
