File: PCB(beta)/PCB(beta).sch (EAGLE design)
At the start: 316 parts, among them IC1 FT232RQ, J1 5.5x2.1mm Barrel, J4 FEMALE 2x3, J6 SSM-120-S-DV, J7 SSM-120-S-DV, J9 DM3AT-SF-PEJM5, K1 692122030100, P1 1-2295018-2, U1 TPS2553DBVT, U10 LSF0108RKSR, U11 LSF0108RKSR, U12 LSF0108RKSR, U2 TLV62084DSGR, U3 LSF0108RKSR, U4 LSF0108RKSR, U5 LSF0108RKSR, U6 LSF0108RKSR, U7 LSF0108RKSR, U8 LSF0108RKSR, U9 LSF0108RKSR

Commit message: complete.
Parts:
- added C100, C101, C102, C109, C110, C111, C112, C113, C114, C115, C116, C117, C118, C119, C120, C121, C122, C123, C124, C125, C126, C127: 0.1uF, SparkFun-Capacitors:0.1UF-0603-25V-(+80/-20%)
- added C103, C104: 1.0uF, SparkFun-Capacitors:1.0UF-0603-16V-10%
- added C105, C106, C107, C108, C128, C129: 10uF, SparkFun-Capacitors:10UF-0603-6.3V-20%
- added R109, R110, R111, R112, R113, R114, R115, R119, R120: 10k, SparkFun-Resistors:10KOHM-0603-1/10W-1%
- added R116: 4.99k, SparkFun-Resistors:4.7KOHM-0603-1/10W-1%
- added R117, R118: 2.7k, SparkFun-Resistors:2.55KOHM-0603-1/10W-1%
- added U$54: PS8203TQFN32GTR-A3, temp:PS8203TQFN32GTR-A3
- added U$55, U$56: DF40C-100DS-0.4V(51)_100PINCONNECTOR, Joule Expansion Board:DF40C-100DS-0.4V(51)_100PINCONNECTOR
Connections:
- removed net ISK_GPIO_4: U8.A2
- new net +V5P0V_VCONN: C119.1, U$55.P$41
- new net DCIN_EN: R109.1, R111.2, U$54.DCIN_EN
- new net DDI1_CTRL_CLK: R118.1, U$54.SCL_SRC, U$55.P$68
- new net DDI1_CTRL_DAT: R117.1, U$54.SDA_SRC, U$55.P$70
- new net EQ: R110.1, R112.2, U$54.EQ
- new net HDMI_CEXT: C100.1, U$54.CEXT
- new net HDMI_OB_DAT0_DP: U$54.OUT_D0P
- new net HDMI_OB_HPD_INV: U$54.HPD_SNK
- new net HDMI_PRE: R119.1, R120.2, U$54.PRE
- new net HDMI_REXT: R116.2, U$54.REXT
- new net INTD_DSI_TE_1: U$56.P$82
- new net ISH_GPIO_4: U$55.P$29, U8.A2
- new net LS_CFG: R114.1, R115.2, U$54.CFG
- new net LS_PD_N: R113.1, U$54.PD*
- new net MDSI_A_CLK_DN: U$56.P$27
- new net MDSI_A_CLK_DP: U$56.P$25
- new net MDSI_A_DATA_0_DN: U$56.P$19
- new net MDSI_A_DATA_0_DP: U$56.P$21
- new net MDSI_A_DATA_1_DN: U$56.P$31
- new net MDSI_A_DATA_1_DP: U$56.P$33
- new net MDSI_A_DATA_2_DN: U$56.P$37
- new net MDSI_A_DATA_2_DP: U$56.P$39
- new net MDSI_A_DATA_3_DN: U$56.P$76
- new net MDSI_A_DATA_3_DP: U$56.P$78
- new net N$41: U$56.P$79
- new net N$74: U$56.P$92
- new net N$75: U$56.P$94
- new net N$76: U$56.P$98
- new net N$77: U$56.P$100
- new net PCIE1_CLKREQ_N: U$56.P$50
- new net PCIE1_CLK_DN: U$56.P$88
- new net PCIE1_CLK_DP: U$56.P$86
- new net PCIE1_PERST_N: U$56.P$70
- new net PCIE1_WAKE_N: U$56.P$72
- new net USB2_ID_PMIC: U$55.P$20
- net +1.8V: now also C102.1, C104.1, R117.2, R118.2, U$54.VDDIO
- net +3V3: now also C101.1, C103.1, R109.2, R110.2, R113.2, R114.2, R119.2, U$54.VDD
- net +VBATTERY: now also C123.1, U$55.P$92
- net +VBUS: now also C120.1, U$55.P$99
- net +VDC_IN: now also C118.1, U$55.P$37
- net +VDD1: now also C122.1, U$55.P$36
- net +VDD3: now also C121.1, U$55.P$30
- net +VRTC: now also C117.1, U$55.P$11
- net +VSYS: now also C105.1, C106.1, C107.1, C108.1, C109.1, C110.1, C111.1, C112.1, C113.1, C114.1, C115.1, C116.1, U$55.P$12, U$55.P$15, U$55.P$17, U$55.P$2, U$55.P$5, U$55.P$7
- net AVS_M_CLK_A1: now also U$56.P$52
- net AVS_M_CLK_B1: now also U$56.P$62
- net AVS_M_DATA_1: now also U$56.P$66
- net BLDRW_0_PWM: now also U$56.P$56
- net BTN_N: now also U$55.P$84
- net CHRG_EN_N: now also U$55.P$35
- net CHRG_INT_N: now also U$55.P$40
- net CLK_19P2M: now also U$55.P$71
- net CODEC_MCLK: now also U$55.P$43
- net DISPLAY_0_BIAS_EN: now also U$56.P$64
- net DISPLAY_0_BKLT_EN: now also U$56.P$58
- net DISPLAY_0_RST_N: now also U$56.P$68
- net FLASH_RST_N: now also U$56.P$71
- net FLASH_TORCH: now also U$56.P$73
- net FLASH_TRIGGER: now also U$56.P$69
- net GND: now also C100.2, C101.2, C102.2, C103.2, C104.2, C105.2, C106.2, C107.2, C108.2, C109.2, C110.2, C111.2, C112.2, C113.2, C114.2, C115.2, C116.2, C117.2, C118.2, C119.2, C120.2, C121.2, C122.2, C123.2, C124.2, C125.2, C126.2, C127.2, C128.2, C129.2, R111.1, R112.1, R115.1, R120.1, U$54.EPAD, U$54.GND, U$55.P$10, U$55.P$100, U$55.P$19, U$55.P$48, U$55.P$54, U$55.P$60, U$55.P$66, U$55.P$72, U$55.P$75, U$55.P$82, U$55.P$86, U$55.P$96, U$55.P$98, U$56.P$10, U$56.P$16, U$56.P$17, U$56.P$2, U$56.P$23, U$56.P$24, U$56.P$29, U$56.P$30, U$56.P$35, U$56.P$36, U$56.P$41, U$56.P$42, U$56.P$48, U$56.P$5, U$56.P$54, U$56.P$60, U$56.P$61, U$56.P$67, U$56.P$74, U$56.P$8, U$56.P$80, U$56.P$84, U$56.P$85, U$56.P$90, U$56.P$91, U$56.P$93, U$56.P$96, U$56.P$99
- net GPIO_22: now also U$55.P$94
- net HDMI_CLK_C_DN: now also U$54.IN_CKN
- net HDMI_CLK_C_DP: now also U$54.IN_CKP
- net HDMI_CLK_DN: now also U$55.P$46
- net HDMI_CLK_DP: now also U$55.P$44
- net HDMI_OB_CLK_DN: now also U$54.OUT_CKN
- net HDMI_OB_CLK_DP: now also U$54.OUT_CKP
- net HDMI_OB_DAT0_DN: now also U$54.OUT_D0N
- net HDMI_OB_DAT1_DN: now also U$54.OUT_D1N
- net HDMI_OB_DAT1_DP: now also U$54.OUT_D1P
- net HDMI_OB_DAT2_DN: now also U$54.OUT_D2N
- net HDMI_OB_DAT2_DP: now also U$54.OUT_D2P
- net HDMI_OB_SCL: now also U$54.SCL_SNK
- net HDMI_OB_SDA: now also U$54.SDA_SNK
- net HDMI_TX_0_C_DN: now also U$54.IN_D0N
- net HDMI_TX_0_C_DP: now also U$54.IN_D0P
- net HDMI_TX_0_DN: now also U$55.P$62
- net HDMI_TX_0_DP: now also U$55.P$64
- net HDMI_TX_1_C_DN: now also U$54.IN_D1N
- net HDMI_TX_1_C_DP: now also U$54.IN_D1P
- net HDMI_TX_1_DN: now also U$55.P$58
- net HDMI_TX_1_DP: now also U$55.P$56
- net HDMI_TX_2_C_DN: now also U$54.IN_D2N
- net HDMI_TX_2_C_DP: now also U$54.IN_D2P
- net HDMI_TX_2_DN: now also U$55.P$50
- net HDMI_TX_2_DP: now also U$55.P$52
- net HPD_SRC: now also U$55.P$65
- net HPD_SRC_N: now also U$54.HPD_SRC
- net I2C_0_SCL: now also U$55.P$57
- net I2C_0_SDA: now also U$55.P$95
- net I2C_1_SCL: now also U$56.P$43
- net I2C_1_SDA: now also U$56.P$45
- net I2C_2_SCL: now also U$56.P$28
- net I2C_2_SDA: now also U$56.P$26
- net I2S_1_CLK: now also U$55.P$39
- net I2S_1_FS: now also U$55.P$45
- net I2S_1_RXD: now also U$55.P$47
- net I2S_1_TXD: now also U$55.P$49
- net ISH_GPIO_0: now also U$55.P$25
- net ISH_GPIO_1: now also U$55.P$27
- net ISH_GPIO_2: now also U$55.P$32
- net ISH_GPIO_3: now also U$55.P$34
- net ISH_GPIO_5: now also U$55.P$38
- net ISH_GPIO_6: now also U$55.P$31
- net ISH_I2C_0_SCL: now also U$55.P$16
- net ISH_I2C_0_SDA: now also U$55.P$18
- net ISH_I2C_1_SCL: now also U$55.P$21
- net ISH_I2C_1_SDA: now also U$55.P$23
- net ISH_UART_0_CTS: now also U$56.P$9
- net ISH_UART_0_RTS: now also U$56.P$11
- net ISH_UART_0_RXD: now also U$56.P$13
- net ISH_UART_0_TXD: now also U$56.P$15
- net OTG_EN: now also U$55.P$69
- net PMIC_PWRBTN_N: now also U$55.P$9
- net PMIC_PWRGOOD: now also U$55.P$33
- net PMIC_RESET_N: now also U$55.P$13
- net PMIC_SLPCLK_1: now also U$56.P$7
- net PWM_0: now also U$55.P$1
- net PWM_1: now also U$55.P$3
- net PWM_2: now also U$55.P$22
- net PWM_3: now also U$55.P$24
- net SDCARD_CD_N: now also U$55.P$79
- net SDCARD_CLK: now also U$55.P$73
- net SDCARD_CMD: now also U$55.P$89
- net SDCARD_D0: now also U$55.P$81
- net SDCARD_D1: now also U$55.P$83
- net SDCARD_D2: now also U$55.P$85
- net SDCARD_D3: now also U$55.P$87
- net SDCARD_LVL_CLK_FB: now also U$55.P$67, U$55.P$77
- net SDCARD_LVL_CMD_DIR: now also U$55.P$90
- net SDCARD_LVL_SEL: now also U$55.P$88
- net SDCARD_PWR_DOWN_N: now also U$55.P$91
- net SPI_0_CLK: now also U$56.P$59
- net SPI_0_FS0: now also U$56.P$75
- net SPI_0_FS1: now also U$56.P$77
- net SPI_0_FS2: now also U$56.P$53
- net SPI_0_MISO: now also U$56.P$49
- net SPI_0_MOSI: now also U$56.P$57
- net SPI_1_CLK: now also U$55.P$53
- net SPI_1_FS0: now also U$55.P$55
- net SPI_1_FS2: now also U$55.P$14
- net SPI_1_MISO: now also U$55.P$63
- net SPI_1_MOSI: now also U$55.P$51
- net UART_0_CTS: now also U$56.P$47
- net UART_0_RTS: now also U$56.P$55
- net UART_0_RXD: now also U$56.P$51
- net UART_0_TXD: now also U$55.P$93
- net UART_1_RXD: now also U$55.P$26
- net UART_1_TXD: now also U$55.P$28
- net UART_2_CTS: now also U$55.P$74
- net UART_2_RTS: now also U$55.P$76
- net UART_2_RXD: now also U$55.P$80
- net UART_2_TXD: now also U$55.P$78
- net USB2_0_DN: now also U$55.P$8
- net USB2_0_DP: now also U$55.P$6
- net USB2_1_DN: now also U$56.P$63
- net USB2_1_DP: now also U$56.P$65
- net USB3_0_RX_DN: now also U$56.P$44
- net USB3_0_RX_DP: now also U$56.P$46
- net USB3_0_TX_DN: now also U$56.P$6
- net USB3_0_TX_DP: now also U$56.P$4
- net USB3_1_RX_DN: now also U$56.P$97
- net USB3_1_RX_DP: now also U$56.P$95
- net USB3_1_TX_DN: now also U$56.P$89
- net USB3_1_TX_DP: now also U$56.P$87
- net USBC_SEL: now also U$56.P$18
- net USB_TYPC_CC1: now also U$55.P$59
- net USB_TYPC_CC2: now also U$55.P$61
- net V+: now also C124.1, C125.1, C126.1, C127.1, C128.1, C129.1, U$56.P$1, U$56.P$20, U$56.P$22, U$56.P$3, U$56.P$32, U$56.P$34
- net VCONN_DCDC_EN: now also U$55.P$97

Commit message: 04/08/2017
Parts:
- added C130, C131: 22pF, SparkFun-Capacitors:22PF-0603-50V-5%
- added C132, C133, C137, C138, C140, C141, C142, C143, C144, C145, C146, C147, C148, C149, C150, C151, C152, C153, C154, C157, C158, C159, C160, C161, C162, C163, C164, C169, C170, C171, C172: 0.1uF, SparkFun-Capacitors:0.1UF-0603-25V-(+80/-20%)
- added C134, C135: 18pF, SparkFun-Capacitors:18PF-0603-50V-5%
- added C136: 1.0uF, SparkFun-Capacitors:1.0UF-0603-16V-10%
- added C139, C155, C156: 10uF, SparkFun-Capacitors:10UF-0603-6.3V-20%
- added C165, C166, C167, C168: 1nF, SparkFun-Capacitors:1.0NF/1000PF-0603-50V-10%
- added C173, C175: 4.7uF, SparkFun-Capacitors:4.7UF0603
- added C174: 10nF, SparkFun-Capacitors:10NF-0603-50V-10%
- added FB10, FB6, FB7, FB8, FB9: 30Ω/1.8A, SparkFun-Coils:FERRITE_BEAD-0603
- added J10: (no value), SparkFun-Connectors:CONN_03X2FEMALE_SMD
- added K2, K3, K4, K5: 692112030100, Joule Expansion Board:692112030100
- added Q3, Q4: 220mA/50V/3.5Ω, SparkFun-DiscreteSemi:MOSFET-NCH-BSS138
- added R121, R122, R123, R124, R125, R131: 10k, SparkFun-Resistors:10KOHM-0603-1/10W-1%
- added R126, R138, R139, R140, R141: 1M, SparkFun-Resistors:1MOHM-0603-1/4W-5%
- added R127, R128, R130, R132, R134, R135, R136, R137: 4.7k, SparkFun-Resistors:4.7KOHM-0603-1/10W-1%
- added R129: 9.53k, SparkFun-Resistors:9.76KOHM-0603-1/10W-1%
- added R133: 90.9k, SparkFun-Resistors:100KOHM-0603-1/10W-1%
- added S4: (no value), SparkFun-Switches:MOMENTARY-SWITCH-SPST-2-SMD-4.6X2.8MM
- added U$57: TUSB8041, Joule Expansion Board:TUSB8041
- added U$58: ADP1706ARDZ-1.1-R7, Joule Expansion Board:ADP1706ARDZ-1.1-R7
- added U13: ATMEGA328P_TQFP, SparkFun-IC-Microcontroller:ATMEGA328P_TQFP
- added Y1: 16MHz, SparkFun-Clocks:CRYSTAL-16MHZSMD-5X3.2
- added Y2: 24MHz, SparkFun-Clocks:CRYSTAL-24MHZ"
- K1: value 692122030100 -> 692112030100; device Wuerth_Elektronik_eiCan_Communication_Connectors_STENCIL:692122030100 -> Joule Expansion Board:692112030100
Connections:
- new net +1V1: C148.1, C149.1, C150.1, C151.1, C152.1, C153.1, C154.1, C155.1, U$57G$2.VDD1, U$57G$2.VDD2, U$57G$2.VDD3, U$57G$2.VDD4, U$57G$2.VDD5, U$57G$2.VDD6, U$57G$2.VDD7, U$57G$2.VDD8
- new net +3V3_HUB: C156.1, C157.1, C158.1, C159.1, C160.1, FB6.1
- new net DM_UP: U$57G$1.USB_DM_UP
- new net DN1_VBUS: FB7.1
- new net DN2_VBUS: FB8.1
- new net DN3_VBUS: FB9.1
- new net DN4_VBUS: FB10.1
- new net DP_UP: U$57G$1.USB_DP_UP
- new net GRST#: C136.1, U$57G$1.GRST#
- new net MICRO_RST: J10.5, R121.1, S4.3, S4.4, U13.PC6(/RESET)
- new net N$10: Q3.D, R123.1, U13.PD0(RXD)
- new net N$15: C132.1, U13.AREF
- new net N$18: R127.2, U$57G$1.TEST
- new net N$2: J10.4, U13.PB3(MOSI/OC2)
- new net N$20: R129.2, U$57G$1.USB_R1
- new net N$21: Q4.D, R124.1, U13.PD1(TXD)
- new net N$22: R132.2, U$57G$1.AUTOEN_HS_SUSPD
- new net N$23: R128.2, U$57G$1.GANGED/SMBA2/HS_UP
- new net N$24: R130.2, U$57G$1.FPMGT/SMBA1/SS_UP
- new net N$25: R131.2, R133.2, U$57G$1.USB_VBUS
- new net N$26: C140.1, U$57G$1.USB_SSTXM_DN4
- new net N$27: C141.1, U$57G$1.USB_SSTXP_DN4
- new net N$28: C142.1, U$57G$1.USB_SSTXM_DN3
- new net N$29: C143.1, U$57G$1.USB_SSTXP_DN3
- new net N$3: J10.1, U13.PB4(MISO)
- new net N$30: C144.1, U$57G$1.USB_SSTXM_DN2
- new net N$31: C145.1, U$57G$1.USB_SSTXP_DN2
- new net N$32: C147.1, U$57G$1.USB_SSTXM_DN1
- new net N$33: C146.1, U$57G$1.USB_SSTXP_DN1
- new net N$34: C148.2, C149.2, C150.2, C151.2, C152.2, C153.2, C154.2, C155.2
- new net N$35: C161.1, FB7.2, K2.VBUS
- new net N$36: C174.1, U$58.SS
- new net N$38: C162.1, FB8.2
- new net N$40: C163.1, FB9.2, K4.VBUS
- new net N$6: J10.3, U13.PB5(SCK)
- new net N$7: C130.2, U13.PB6(XTAL1/TOSC1), Y1.2
- new net N$73: C164.1, FB10.2, K5.VBUS
- new net N$9: C131.2, U13.PB7(XTAL2/TOSC2), Y1.1
- new net OVERCUR1Z: U$57G$1.OVERCURZ1
- new net OVERCURZ2: U$57G$1.OVERCURZ2
- new net OVERCURZ3: U$57G$1.OVERCURZ3
- new net OVERCURZ4: U$57G$1.OVERCURZ4
- new net PWRCTL1_BATEN1: R134.1, U$57G$1.PWRCTL1/BATEN1
- new net PWRCTL2_BATEN2: R135.1, U$57G$1.PWRCTL2/BATEN2
- new net PWRCTL3_BATEN3: R136.1, U$57G$1.PWRCTL3/BATEN3
- new net PWRCTL4-BATEN4: R137.1, U$57G$1.PWRCTL4/BATEN4
- new net SSRXM_UP: U$57G$1.USB_SSRXM_UP
- new net SSRXP_UP: U$57G$1.USB_SSRXP_UP
- new net USB_DM_DN1: K2.D-, U$57G$1.USB_DM_DN1
- new net USB_DM_DN2: K3.D-, U$57G$1.USB_DM_DN2
- new net USB_DM_DN3: K4.D-, U$57G$1.USB_DM_DN3
- new net USB_DM_DN4: K5.D-, U$57G$1.USB_DM_DN4
- new net USB_DP_DN1: K2.D+, U$57G$1.USB_DP_DN1
- new net USB_DP_DN2: K3.D+, U$57G$1.USB_DP_DN2
- new net USB_DP_DN3: K4.D+, U$57G$1.USB_DP_DN3
- new net USB_DP_DN4: K5.D+, U$57G$1.USB_DP_DN4
- new net USB_SSRXM_DN1: K2.STDA_SSRX-, U$57G$1.USB_SSRXM_DN1
- new net USB_SSRXM_DN2: K3.STDA_SSRX-, U$57G$1.USB_SSRXM_DN2
- new net USB_SSRXM_DN3: K4.STDA_SSRX-, U$57G$1.USB_SSRXM_DN3
- new net USB_SSRXM_DN4: K5.STDA_SSRX-, U$57G$1.USB_SSRXM_DN4
- new net USB_SSRXP_DN1: K2.STDA_SSRX+, U$57G$1.USB_SSRXP_DN1
- new net USB_SSRXP_DN2: K3.STDA_SSRX+, U$57G$1.USB_SSRXP_DN2
- new net USB_SSRXP_DN3: K4.STDA_SSRX+, U$57G$1.USB_SSRXP_DN3
- new net USB_SSRXP_DN4: K5.STDA_SSRX+, U$57G$1.USB_SSRXP_DN4
- new net USB_SSTXM_DN1: C147.2, K2.STDA_SSTX-
- new net USB_SSTXM_DN2: C144.2, K3.STDA_SSTX-
- new net USB_SSTXM_DN3: C142.2, K4.STDA_SSTX-
- new net USB_SSTXM_DN4: C140.2, K5.STDA_SSTX-
- new net USB_SSTXM_UP: C138.1
- new net USB_SSTXP_DN1: C146.2, K2.STDA_SSTX+
- new net USB_SSTXP_DN2: C145.2, K3.STDA_SSTX+
- new net USB_SSTXP_DN3: C143.2, K4.STDA_SSTX+
- new net USB_SSTXP_DN4: C141.2, K5.STDA_SSTX+
- new net USB_SSTXP_UP: C137.1
- new net VBUS_HUB: C139.1, R133.1
- new net X: C137.2, U$57G$1.USB_SSTXP_UP
- new net XI: C135.2, R126.2, U$57G$1.XI, Y2.2
- new net XO: C134.2, R126.1, U$57G$1.XO, Y2.1
- new net Y: C138.2, U$57G$1.USB_SSTXM_UP
- net +3V3: now also C173.1, FB6.2, Q3.G, Q4.G, R122.2, R125.2, R134.2, R135.2, R136.2, R137.2, U$58.EN, U$58.IN, U$58.IN2
- net +5V: now also C133.1, J10.2, R121.2, R123.2, R124.2, U13.AVCC, U13.VCC@4, U13.VCC@6
- net GND: now also C130.1, C131.1, C132.2, C133.2, C134.1, C135.1, C136.2, C139.2, C156.2, C157.2, C158.2, C159.2, C160.2, C161.2, C162.2, C163.2, C164.2, C165.1, C165.2, C166.1, C166.2, C167.1, C167.2, C168.1, C168.2, C169.1, C169.2, C170.1, C170.2, C171.1, C171.2, C172.1, C172.2, C173.2, C174.2, C175.2, J10.6, K2.GND, K2.GND_DRAIN, K3.GND, K3.GND_DRAIN, K4.GND, K5.GND, R127.1, R128.1, R129.1, R130.1, R131.1, R132.1, R138.1, R138.2, R139.1, R139.2, R140.1, R140.2, R141.1, R141.2, S4.1, S4.2, U$57G$2.PAD, U$57G$2.VDD33_1, U$57G$2.VDD33_2, U$57G$2.VDD33_3, U$57G$2.VDD33_4, U$58.GND, U13.AGND, U13.GND@3, U13.GND@5
- net UART_0_RXD_LS: now also Q4.S, R125.1
- net UART_0_TXD_LS: now also Q3.S, R122.1
- net V+: now also C175.1, U$58.OUT, U$58.OUT2, U$58.SENSE

Commit message: 04/10/2017
Parts:
- removed K1: 692112030100, Joule Expansion Board:692112030100
- added C176, C177, C180, C181, C182, C184, C186: 0.1uF, SparkFun-Capacitors:0.1UF-0603-25V-(+80/-20%)
- added C178, C179, C183, C185: 150uF, SparkFun-Capacitors:100UF-POLAR-RADIAL-2.5MM-25V-20%
- added R142, R145: 25.5k, SparkFun-Resistors:26.7KOHM0603-1/10W-1%
- added R143, R144, R146, R147: 10k, SparkFun-Resistors:10KOHM-0603-1/10W-1%
- added U$59, U$60: TPS2561DRCT, Joule Expansion Board:TPS2561DRCT
- added U14: 433MHz, SparkFun-RF:RFM69HCW-433
- added U15: SN74LVC1G373DCKR, Texas Instruments_By_element14_Batch_1:SN74LVC1G373DCKR
Connections:
- removed net DM_UP: U$57G$1.USB_DM_UP
- removed net DP_UP: U$57G$1.USB_DP_UP
- removed net OVERCURZ2: U$57G$1.OVERCURZ2
- removed net OVERCURZ3: U$57G$1.OVERCURZ3
- removed net OVERCURZ4: U$57G$1.OVERCURZ4
- removed net PWRCTL4-BATEN4: R137.1, U$57G$1.PWRCTL4/BATEN4
- removed net SSRXM_UP: U$57G$1.USB_SSRXM_UP
- removed net SSRXP_UP: U$57G$1.USB_SSRXP_UP
- removed net USB_SSTXM_UP: C138.1
- removed net USB_SSTXP_UP: C137.1
- new net ILIM1: R142.2, U$59.ILIM
- new net ILIM2: R145.2, U$60.ILIM
- new net N$45: C184.1, C185.+, U$60.OUT2
- new net OVERCUR2Z: R144.1, U$57G$1.OVERCURZ2, U$59.FAULT2Z
- new net OVERCUR3Z: R146.1, U$57G$1.OVERCURZ3, U$60.FAULT1Z
- new net OVERCUR4Z: R147.1, U$57G$1.OVERCURZ4, U$60.FAULT2Z
- new net PWRCTL4_BATEN4: R137.1, U$57G$1.PWRCTL4/BATEN4, U$60.EN2
- net +1V1: now also C175.1, U$58.OUT, U$58.OUT2, U$58.SENSE
- net +3V3: now also C186.1, C81.1, R143.2, R144.2, R146.2, R147.2, U14.3.3V, U15.VCC
- net +5V: now also C176.1, C177.1, U$59.IN, U$59.IN2, U$60.IN, U$60.IN2
- net +V5P0V_USBA: no longer C81.1, K1.VBUS
- net DN1_VBUS: now also C178.+, C180.1, U$59.OUT1
- net DN2_VBUS: now also C179.+, C181.1, U$59.OUT2
- net DN3_VBUS: now also C182.1, C183.+, U$60.OUT1
- net GND: now also C176.2, C177.2, C178.-, C179.-, C180.2, C181.2, C182.2, C183.-, C184.2, C185.-, C186.2, R142.1, R145.1, U$59.GND, U$59.PAD, U$60.GND, U$60.PAD, U15.GND; no longer K1.GND, K1.GND_DRAIN
- net OVERCUR1Z: now also R143.1, U$59.FAULT1Z
- net PWRCTL1_BATEN1: now also U$59.EN1
- net PWRCTL2_BATEN2: now also U$59.EN2
- net PWRCTL3_BATEN3: now also U$60.EN1
- net USBA_USB2_1_DN: now also U$57G$1.USB_DM_UP; no longer K1.D-
- net USBA_USB2_1_DP: now also U$57G$1.USB_DP_UP; no longer K1.D+
- net USBA_USB3_1_RX_DN: now also U$57G$1.USB_SSRXM_UP; no longer K1.STDA_SSRX-, K1.STDA_SSTX-
- net USBA_USB3_1_RX_DP: now also U$57G$1.USB_SSRXP_UP; no longer K1.STDA_SSRX+, K1.STDA_SSTX+
- net USBA_USB3_1_TX_DN: now also C138.1
- net USBA_USB3_1_TX_DP: now also C137.1
- net V+: no longer C175.1, U$58.OUT, U$58.OUT2, U$58.SENSE
