File: PCB/Chaos/Joulev2_RealTime.brd (EAGLE design)
At the start: 85 x 70 mm, 127 parts, among them IC2 LM340S-12, IC3 LM340S-12, J1 2-PIN_2MM-V, K1 692112030100, K2 692112030100, K3 692112030100, K4 692112030100, K5 692112030100, Q1 N_CH_MOSFET_FDLBL260N100, U1 ATMEGA328P_TQFP, U2 74VHC_MUXSO16, U3 RFM69CW, U4 TUSB8041, U5 ADP1706ARDZ-1.1-R7, U6 TPS2561DRCT, U7 TPS2561DRCT, U8 ATTINY441/841SSU/SSUR, U9 TXB0108PWR, X1 J12HEADER_(JOULE), X2 J13HEADER_(JOULE), X4 TRAXXAS-CON, Y1 16MHz, Y2 24MHz

Commit message: 'fixed' chaos
Parts:
- U8: value ATTINY441/841SSU/SSUR -> (none)
- moved R1 190.8 mm to (74.9, 29.7)
- moved U2 185.3 mm to (73.7, 23.2), turned to 270 degrees
- moved C3 181.2 mm to (70.0, 63.9), turned to 90 degrees
- moved C2 180.3 mm to (73.2, 65.0)
- moved C1 175.7 mm to (73.2, 68.2)
- moved S1 173.6 mm to (81.2, 25.7)
- moved JP5 172.8 mm to (80.6, 41.0), flipped to the bottom
- moved JP6 169.3 mm to (82.6, 19.1)
- moved C29 167.5 mm to (36.9, 7.48), turned to 180 degrees
- moved JP4 165.3 mm to (80.6, 38.4), flipped to the bottom
- moved U3 161.5 mm to (74.6, 8.90)
- moved JP3 158.0 mm to (80.6, 35.9), flipped to the bottom
- moved D1 157.1 mm to (30.1, 18.5), turned to 270 degrees
- moved C56 155.5 mm to (30.1, 22.2)
- moved U1 153.6 mm to (60.1, 18.4)
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Connections:
- net V3P3V renamed S$2
- removed net ACHANNEL_5V: IMU.2
- removed net BCHANNEL_5V: IMU.4
- removed net DIO0_3V3: U3.9, U8.10
- removed net ESTOP_3V3: U8.3, U9.5
- removed net ESTOP_5V: J1.1, U9.16
- removed net MISO_3V3: U3.8
- removed net MISO_JOULE: U9.8
- removed net MODE_SELECT_3V3: U8.11
- removed net MOSI_3V3: U3.5
- removed net MOSI_JOULE: U9.7
- removed net N$12: R43.1, U8.4
- removed net N$13: C59.1, U1.20
- removed net NSS_JOULE: U9.6
- removed net RC_CH3_3V3: U8.12
- removed net RC_CH3_5V: JP1.3
- removed net SCK_3V3: U3.6
- removed net SCK_5V: U1.17, U9.12
- removed net SCK_JOULE: U9.9
- new net DIO0_3P3V: U3.9
- new net DIO0_5V: U1.32
- new net ESTOP: J1.1, U1.2
- new net RC_MODE: JP1.3, U1.11
- net 3.3V: no longer ENCODER.2, IC2.3, R43.2, U8.1, U9.2
- net 5V: no longer C60.1, IC2.1, IC3.3, IMU.1, U9.19
- net 5V_MODE_SELECT: now also U1.12
- net GND: no longer C59.2, C60.2, C61.2, ENCODER.1, IC2.TAB, IC3.TAB, IMU.3, JP5.1, U8.14, U9.11
- net I2C0_SCL: no longer ENCODER.4
- net I2C0_SDA: no longer ENCODER.3
- net MISO_3P3V: now also U3.8
- net MISO_5V: no longer U9.13
- net MOSI_3P3V: now also U3.5
- net MOSI_5V: no longer U9.14
- net N$5: now also Q1.DRAIN; no longer TRAXXAS_ESC_PWR.GND
- net NSS_5V: no longer U9.15
- net SCK_3P3V: now also U3.6
- net VCC: no longer C61.1, IC3.1, TRAXXAS_ESC_PWR.V+
Routing:
- net N$13: track 0.00 -> 4.50 mm
