File: PCB/Joulev2_RealTime.brd (EAGLE design)
At the start: 86 x 72.5 mm, 120 parts, among them IC3 LM340S-05, J1 2-PIN_2MM-V, Q1 N_CH_MOSFET_FDLBL260N100, U1 ATMEGA328P_TQFP, U2 74VHC_MUXSO16, U3 RFM69CW, U4 ADP1706ARDZ-1.1-R7, U5 TPS2561DRCT, U6 TPS2561DRCT, U8 ATTINY441/841SSU/SSUR, U9 TXB0108PWR, X1 J12HEADER_(JOULE), X2 J13HEADER_(JOULE), X4 TRAXXAS-CON, Y1 16MHz, Y2 24MHz

Commit message: night.
Parts:
- added R29: 10, rcl:R0603
- added U$9: (no value), Roboracing:SOT363
- moved C49 94.2 mm to (67.5, 17.0), turned to 270 degrees
- moved R27 82.4 mm to (56.0, 16.5), turned to 180 degrees
- moved C48 81.0 mm to (56.0, 19.0), turned to 180 degrees
- moved C47 79.1 mm to (55.0, 22.0), turned to 270 degrees
- moved C45 61.9 mm to (46.5, 22.0), turned to 270 degrees
- moved C46 57.1 mm to (44.0, 22.0), turned to 270 degrees
- moved C44 55.4 mm to (49.0, 22.0), turned to 270 degrees
- moved U4 54.8 mm to (48.0, 26.5), turned to 90 degrees
- moved C38 1.15 mm to (18.0, 26.2), turned to 90 degrees
- moved C3 1.12 mm to (57.5, 22.0), turned to 270 degrees
- moved C60 0.56 mm to (55.5, 11.8)
- moved R26 0.50 mm to (15.1, 26.3)
- moved C36 0.50 mm to (19.1, 22.7)
- moved C39 0.50 mm to (21.6, 22.7)
- moved R5 0.50 mm to (21.0, 17.9)
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Routing:
- net 1.1V: track 53.9 -> 31.4 mm
- net 3.3V: track 78.1 -> 92.4 mm, vias 5 -> 8
- net GND: track 193.1 -> 201.5 mm, vias 63 -> 69
- net N$41: track 0.00 -> 5.94 mm
- net 5V: track 107.9 -> 109.8 mm
- net N$30: track 12.0 -> 13.4 mm
- net N$32: track 61.3 -> 60.4 mm
- net N$34: track 63.7 -> 62.7 mm
- net I2C0_SCL: track 66.6 -> 67.3 mm
- net DN3_VBUS: track 40.3 -> 40.9 mm
- net OVERCUR2Z: track 15.3 -> 15.9 mm
- net N$26: track 4.01 -> 3.43 mm
- net N$29: track 9.24 -> 9.77 mm

Commit message: Fixed f/b, more routing
Parts:
- removed U$9: (no value), Roboracing:SOT363
- added U10: ZXGD3009DY, Roboracing:SOT363
- moved R29 121.9 mm to (72.2, 70.0), turned to 270 degrees
- moved Q1 4.00 mm to (66.4, 66.0)
- moved R2 2.55 mm to (74.4, 68.0), flipped to the top
- moved D1 0.56 mm to (56.0, 3.50), turned to 90 degrees
Connections:
- new net N$42: R29.1, U10.4, U10.6
- new net N$43: Q1.GATE, R2.1, R29.2
- net 5V: now also U10.1
- net ESTOP_GATE: now also U10.2; no longer Q1.GATE, R2.1
- net GND: now also U10.3
Routing:
- net 3.3V: track 92.4 -> 173.7 mm, vias 8 -> 13
- net 5V: track 109.8 -> 180.2 mm, vias 6 -> 13
- net N$43: track 0.00 -> 6.07 mm
- net GND: track 201.5 -> 207.2 mm
- net N$42: track 0.00 -> 4.54 mm
- net N$5: track 8.82 -> 12.8 mm
- net ESTOP_GATE: track 8.23 -> 4.80 mm

Commit message: done?
Parts:
- added U$9: (no value), RoboJackets-Aesthetics:ROBOBUZZ_0.6X
- moved ENCODER 81.3 mm to (3.15, 60.7)
- moved IMU 12.5 mm to (83.7, 49.2)
- moved X1 0.32 mm to (35.4, 69.3), turned to 180 degrees
- moved X2 0.32 mm to (35.4, 33.8), turned to 180 degrees
- moved FB1 0.19 mm to (7.06, 30.7)
Connections:
- removed net NSS_5V: U1.14, U9.15
- removed net NSS_JOULE: U9.6
- net 3.3V: now also IMU.2; no longer ENCODER.2
- net 5V: now also ENCODER.1; no longer IMU.1
- net ACHANNEL_5V: now also ENCODER.2, X1.35; no longer IMU.2
- net BCHANNEL_5V: now also ENCODER.4, X1.33; no longer IMU.4
- net GND: now also ENCODER.3, IMU.1; no longer ENCODER.1, IMU.3
- net I2C0_SCL: now also IMU.4; no longer ENCODER.4
- net I2C0_SDA: now also IMU.3; no longer ENCODER.3
Routing:
- net 5V: track 180.2 -> 256.7 mm
- net MISO_JOULE: track 19.8 -> 47.9 mm
- net ACHANNEL_5V: track 0.00 -> 25.4 mm
- net SCK_JOULE: track 27.3 -> 52.2 mm
- net BCHANNEL_5V: track 0.00 -> 24.3 mm
- net MOSI_JOULE: track 27.9 -> 47.8 mm
- net I2C0_SCL: track 67.3 -> 51.6 mm
- net I2C0_SDA: track 69.9 -> 60.2 mm
- net GND: track 207.2 -> 210.5 mm
- net NSS_5V: track 2.67 -> 0.00 mm
- net N$32: track 60.4 -> 61.0 mm
- net N$23: track 3.61 -> 4.13 mm

Commit message: done?
Connections:
- removed net N$7: JP1.2, JP2.2, JP3.2, JP4.2, JP5.2
- net 5V: now also JP1.2, JP2.2, JP3.2, JP4.2, JP5.2
Routing:
- net 5V: track 256.7 -> 273.5 mm
- net N$7: track 10.2 -> 0.00 mm
Changed lines of the file:
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@@
 <wire x1="82.775" y1="62.81" x2="82.765" y2="62.82" width="0.3" layer="3"/>
-</signal>
-<signal name="N$7">
-<contactref element="JP5" pad="2"/>
-<contactref element="JP4" pad="2"/>
-<contactref element="JP1" pad="2"/>
-<contactref element="JP2" pad="2"/>
-<contactref element="JP3" pad="2"/>
-<wire x1="80.47" y1="14.04" x2="80.47" y2="11.5" width="0.3" layer="1"/>
-<wire x1="80.47" y1="11.5" x2="80.47" y2="8.96" width="0.3" layer="1"/>
-<wire x1="80.47" y1="8.96" x2="80.47" y2="6.42" width="0.3" layer="1"/>
-<wire x1="80.47" y1="6.42" x2="80.47" y2="3.88" width="0.3" layer="1"/>
 </signal>
 <signal name="N$20">
@@
 <wire x1="7.41" y1="56.91" x2="3.15" y2="56.91" width="0.3" layer="3"/>
 <wire x1="9" y1="58.5" x2="7.41" y2="56.91" width="0.3" layer="3"/>
-<wire x1="76.5" y1="18" x2="80.55" y2="22.05" width="0.3" layer="3"/>
+<wire x1="76.5" y1="18" x2="78.25" y2="19.75" width="0.3" layer="3"/>
+<wire x1="78.25" y1="19.75" x2="80.55" y2="22.05" width="0.3" layer="3"/>
 <wire x1="80.55" y1="22.05" x2="80.55" y2="50.22781875" width="0.3" layer="3"/>
+<contactref element="JP5" pad="2"/>
+<contactref element="JP4" pad="2"/>
+<contactref element="JP1" pad="2"/>
+<contactref element="JP2" pad="2"/>
+<contactref element="JP3" pad="2"/>
+<wire x1="78.25" y1="19.75" x2="80.47" y2="17.53" width="0.3" layer="3"/>
+<wire x1="80.47" y1="17.53" x2="80.47" y2="14.04" width="0.3" layer="3"/>
+<wire x1="80.47" y1="14.04" x2="80.47" y2="11.5" width="0.3" layer="3"/>
+<wire x1="80.47" y1="11.5" x2="80.47" y2="8.96" width="0.3" layer="3"/>
+<wire x1="80.47" y1="8.96" x2="80.47" y2="6.42" width="0.3" layer="3"/>
+<wire x1="80.47" y1="6.42" x2="80.47" y2="3.88" width="0.3" layer="3"/>
 </signal>
 <signal name="MOSI_JOULE">

Commit message: done? take 2
Parts:
- added R28: 500, rcl:R0603
- moved R2 1.57 mm to (73.0, 67.4), turned to 180 degrees
Connections:
- new net N$7: R28.2, U10.2
- net ESTOP_GATE: now also R28.1; no longer U10.2
Routing:
- net N$7: track 0.00 -> 10.3 mm
- net GND: track 210.5 -> 206.0 mm, vias 69 -> 70
- net ESTOP_GATE: track 4.80 -> 6.73 mm
- net N$43: track 6.07 -> 6.85 mm
Changed lines of the file:
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@@
 <layer number="25" name="tNames" color="7" fill="1" visible="yes" active="yes"/>
 <layer number="26" name="bNames" color="7" fill="1" visible="yes" active="yes"/>
-<layer number="27" name="tValues" color="7" fill="1" visible="no" active="yes"/>
-<layer number="28" name="bValues" color="7" fill="1" visible="no" active="yes"/>
+<layer number="27" name="tValues" color="7" fill="1" visible="yes" active="yes"/>
+<layer number="28" name="bValues" color="7" fill="1" visible="yes" active="yes"/>
 <layer number="29" name="tStop" color="7" fill="3" visible="no" active="yes"/>
 <layer number="30" name="bStop" color="7" fill="6" visible="no" active="yes"/>
@@
 <element name="Q1" library="Roboracing" package="MO-299A" value="N_CH_MOSFET_FDLBL260N100" x="66.38" y="66" smashed="yes" rot="R180">
 <attribute name="NAME" x="68.92" y="58.38" size="0.5" layer="25" font="vector" rot="R180"/>
-<attribute name="VALUE" x="70.19" y="66" size="0.5" layer="25" font="vector" rot="R180"/>
 </element>
 <element name="R1" library="rcl" package="R0603" value="10k" x="62.9" y="2.06" smashed="yes">
@@
 <attribute name="VALUE" x="29.0425" y="18.1775" size="1.27" layer="27" rot="R90"/>
 </element>
-<element name="R2" library="rcl" package="R0603" value="10k" x="74.44" y="68.01" smashed="yes" rot="R270">
-<attribute name="NAME" x="75.1375" y="67.52" size="0.5" layer="25" rot="R270"/>
-<attribute name="VALUE" x="72.535" y="68.645" size="1.27" layer="27" rot="R270"/>
+<element name="R2" library="rcl" package="R0603" value="10k" x="73.01" y="67.3725" smashed="yes" rot="R180">
+<attribute name="NAME" x="72.52" y="66.675" size="0.5" layer="25" rot="R180"/>
+<attribute name="VALUE" x="73.645" y="69.2775" size="1.27" layer="27" rot="R180"/>
 </element>
 <element name="R20" library="rcl" package="R0603" value="25.5k" x="30.67" y="23.9075" smashed="yes">
@@
 </element>
 <element name="U$9" library="RoboJackets-Aesthetics" package="ROBOBUZZ_0.6X" value="" x="47.5" y="8.8125"/>
+<element name="R28" library="rcl" library_urn="urn:adsk.eagle:library:334" package="R0603" value="500" x="73" y="65.3125" rot="R180"/>
 </elements>
 <signals>
@@
 <wire x1="75.4875" y1="72.025" x2="76.3375" y2="72.025" width="0.3" layer="1"/>
 <wire x1="76.3375" y1="72.025" x2="76.75" y2="72.4375" width="0.3" layer="1"/>
-<wire x1="74.44" y1="67.16" x2="71.84" y2="67.16" width="0.3" layer="1"/>
-<wire x1="71.84" y1="67.16" x2="71" y2="68" width="0.3" layer="1"/>
-<wire x1="71" y1="68" x2="70.25" y2="68" width="0.3" layer="1"/>
-<wire x1="70.25" y1="68" x2="69.25" y2="69" width="0.3" layer="1"/>
 <wire x1="11" y1="24.75" x2="10.93" y2="24.68" width="0.3" layer="1"/>
 <wire x1="10.93" y1="24.68" x2="10.93" y2="23.45" width="0.3" layer="1"/>
 <wire x1="12.22" y1="21.5925" x2="11" y2="22.8125" width="0.3" layer="16"/>
 <wire x1="11" y1="22.8125" x2="11" y2="24.75" width="0.3" layer="16"/>
+<wire x1="72.16" y1="67.3725" x2="71.5325" y2="68" width="0.3" layer="1"/>
+<wire x1="71.5325" y1="68" x2="71" y2="68" width="0.3" layer="1"/>
+<via x="71" y="68" extent="1-16" drill="0.35"/>
 </signal>
 <signal name="N$2">
@@
 <wire x1="75.4875" y1="70.0125" x2="75.5" y2="70" width="0.2" layer="1"/>
 <via x="75.5" y="70" extent="1-16" drill="0.35"/>
-<wire x1="75.5" y1="70" x2="75.5" y2="66" width="0.3" layer="3"/>
-<wire x1="75.5" y1="66" x2="75.5" y2="56.5" width="0.3" layer="3"/>
+<wire x1="75.5" y1="56.5" x2="75.5" y2="67" width="0.3" layer="3"/>
 <wire x1="75.5" y1="56.5" x2="76" y2="56" width="0.3" layer="3"/>
 <wire x1="76" y1="56" x2="79.5" y2="56" width="0.3" layer="3"/>
@@
 <wire x1="63.05146875" y1="17.4" x2="63.25146875" y2="17.6" width="0.3" layer="3"/>
 <wire x1="57.5" y1="22.85" x2="58.725" y2="22.85" width="0.3" layer="1"/>
-<wire x1="75.5" y1="66" x2="11" y2="66" width="0.3" layer="3"/>
+<wire x1="74.5" y1="66" x2="11" y2="66" width="0.3" layer="3"/>
 <wire x1="11" y1="66" x2="9" y2="64" width="0.3" layer="3"/>
 <wire x1="9" y1="64" x2="9" y2="58.5" width="0.3" layer="3"/>
@@
 <wire x1="80.47" y1="8.96" x2="80.47" y2="6.42" width="0.3" layer="3"/>
 <wire x1="80.47" y1="6.42" x2="80.47" y2="3.88" width="0.3" layer="3"/>
+<wire x1="75.5" y1="67" x2="75.5" y2="70" width="0.3" layer="3"/>
+<wire x1="74.5" y1="66" x2="75.5" y2="67" width="0.3" layer="3"/>
 </signal>
 <signal name="MOSI_JOULE">
@@
 <signal name="ESTOP_GATE">
 <contactref element="J1" pad="2"/>
-<contactref element="U10" pad="2"/>
-<wire x1="75.4875" y1="71.375" x2="76.505" y2="71.375" width="0.3" layer="1"/>
-<wire x1="76.505" y1="71.375" x2="79.18" y2="68.7" width="0.3" layer="1"/>
+<contactref element="R28" pad="1"/>
+<wire x1="73.85" y1="65.3125" x2="75.7925" y2="65.3125" width="0.3" layer="1"/>
+<wire x1="75.7925" y1="65.3125" x2="79.18" y2="68.7" width="0.3" layer="1"/>
 </signal>
 <signal name="N$9">
@@
 <contactref element="R29" pad="2"/>
 <contactref element="Q1" pad="GATE"/>
-<wire x1="74.15" y1="69.15" x2="72.1875" y2="69.15" width="0.3" layer="1"/>
-<wire x1="74.15" y1="69.15" x2="74.44" y2="68.86" width="0.2" layer="1"/>
-<wire x1="72.1875" y1="69.15" x2="70.58" y2="69.15" width="0.3" layer="1"/>
+<wire x1="70.58" y1="69.15" x2="72.1875" y2="69.15" width="0.3" layer="1"/>
 <wire x1="70.58" y1="69.15" x2="70.58" y2="71.24" width="0.3" layer="1"/>
+<wire x1="72.1875" y1="69.15" x2="73.35" y2="69.15" width="0.3" layer="1"/>
+<wire x1="73.86" y1="68.64" x2="73.86" y2="67.3725" width="0.3" layer="1"/>
+<wire x1="73.35" y1="69.15" x2="73.86" y2="68.64" width="0.3" layer="1"/>
 </signal>
 <signal name="N$44">
 </signal>
+<signal name="N$7">
+<contactref element="U10" pad="2"/>
+<contactref element="R28" pad="2"/>
+<wire x1="72.15" y1="65.3125" x2="72.15" y2="66.0875" width="0.3" layer="1"/>
+<wire x1="72.15" y1="66.0875" x2="72.4375" y2="66.375" width="0.3" layer="1"/>
+<wire x1="72.4375" y1="66.375" x2="75.375" y2="66.375" width="0.3" layer="1"/>
+<wire x1="75.375" y1="66.375" x2="76.5" y2="67.5" width="0.3" layer="1"/>
+<wire x1="76.5" y1="67.5" x2="76.5" y2="70.9375" width="0.3" layer="1"/>
+<wire x1="76.0625" y1="71.375" x2="75.4875" y2="71.375" width="0.3" layer="1"/>
+<wire x1="76.5" y1="70.9375" x2="76.0625" y2="71.375" width="0.3" layer="1"/>
+</signal>
 </signals>

Commit message: done? take 3
Connections:
- removed net ESTOP_GATE: J1.2, R28.1
- new net N$45: J1.2, R29.2
- net ESTOP_5V: now also R28.1; no longer J1.1
- net N$43: now also J1.1; no longer R29.2
Routing:
- net ESTOP_GATE: track 6.73 -> 0.00 mm
- net N$43: track 6.85 -> 4.08 mm
- net ESTOP_5V: track 73.3 -> 70.8 mm
Changed lines of the file:
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@@
 <signal name="ESTOP_5V">
 <contactref element="U9" pad="16"/>
-<contactref element="J1" pad="1"/>
 <wire x1="62.224996875" y1="14.9506" x2="62.224996875" y2="17.724996875" width="0.3" layer="1"/>
 <wire x1="62.224996875" y1="17.724996875" x2="62.5" y2="18" width="0.3" layer="1"/>
@@
 <wire x1="76" y1="64.5" x2="76.5" y2="65" width="0.3" layer="16"/>
 <wire x1="76.5" y1="65" x2="80" y2="65" width="0.3" layer="16"/>
-<wire x1="81.18" y1="66.18" x2="81.18" y2="68.7" width="0.3" layer="16"/>
 <wire x1="80" y1="65" x2="81.18" y2="66.18" width="0.3" layer="16"/>
+<contactref element="R28" pad="1"/>
+<wire x1="76" y1="64.5" x2="73.85" y2="65.3125" width="0" layer="19" extent="1-16"/>
 </signal>
 <signal name="ESTOP_3V3">
@@
 <wire x1="64" y1="30" x2="64" y2="28.23" width="0.3" layer="1"/>
 <wire x1="64" y1="28.23" x2="64.18" y2="28.05" width="0.3" layer="1"/>
-</signal>
-<signal name="ESTOP_GATE">
-<contactref element="J1" pad="2"/>
-<contactref element="R28" pad="1"/>
-<wire x1="73.85" y1="65.3125" x2="75.7925" y2="65.3125" width="0.3" layer="1"/>
-<wire x1="75.7925" y1="65.3125" x2="79.18" y2="68.7" width="0.3" layer="1"/>
 </signal>
 <signal name="N$9">
@@
 <signal name="N$43">
 <contactref element="R2" pad="1"/>
-<contactref element="R29" pad="2"/>
 <contactref element="Q1" pad="GATE"/>
-<wire x1="70.58" y1="69.15" x2="72.1875" y2="69.15" width="0.3" layer="1"/>
 <wire x1="70.58" y1="69.15" x2="70.58" y2="71.24" width="0.3" layer="1"/>
-<wire x1="72.1875" y1="69.15" x2="73.35" y2="69.15" width="0.3" layer="1"/>
 <wire x1="73.86" y1="68.64" x2="73.86" y2="67.3725" width="0.3" layer="1"/>
 <wire x1="73.35" y1="69.15" x2="73.86" y2="68.64" width="0.3" layer="1"/>
+<contactref element="J1" pad="1"/>
+<wire x1="73.86" y1="68.64" x2="81.18" y2="68.7" width="0" layer="19" extent="1-1"/>
+<wire x1="70.58" y1="69.15" x2="73.35" y2="69.15" width="0" layer="19" extent="1-1"/>
 </signal>
 <signal name="N$44">
@@
 <wire x1="76.5" y1="70.9375" x2="76.0625" y2="71.375" width="0.3" layer="1"/>
 </signal>
+<signal name="N$45">
+<contactref element="J1" pad="2"/>
+<contactref element="R29" pad="2"/>
+<wire x1="72.1875" y1="69.15" x2="79.18" y2="68.7" width="0" layer="19" extent="1-1"/>
+</signal>
 </signals>

Commit message: done? take 3
Parts:
- C11, C14, C17, C8: value 1nF -> 1000pF
- moved J1 1.86 mm to (79.3, 68.8), turned to 0 degrees
Routing:
- net N$45: track 0.00 -> 10.1 mm, vias 0 -> 2
- net N$43: track 4.08 -> 12.3 mm, vias 0 -> 2
- net ESTOP_5V: track 70.8 -> 68.1 mm, vias 3 -> 4
Changed lines of the file:
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@@
 <attribute name="VALUE" x="8.595" y="33.585" size="1.27" layer="27" rot="R90"/>
 </element>
-<element name="C11" library="rcl" package="C0603" value="1nF" x="2.33" y="14.12" smashed="yes" rot="MR180">
+<element name="C11" library="rcl" package="C0603" value="1000pF" x="2.33" y="14.12" smashed="yes" rot="MR180">
 <attribute name="NAME" x="1.695" y="13.485" size="0.5" layer="26" rot="MR180"/>
 <attribute name="VALUE" x="1.695" y="16.025" size="1.27" layer="28" rot="MR180"/>
@@
 <attribute name="VALUE" x="9.095" y="14.385" size="1.27" layer="27" rot="R90"/>
 </element>
-<element name="C14" library="rcl" package="C0603" value="1nF" x="10.8" y="3.15" smashed="yes" rot="MR90">
+<element name="C14" library="rcl" package="C0603" value="1000pF" x="10.8" y="3.15" smashed="yes" rot="MR90">
 <attribute name="NAME" x="11.435" y="2.515" size="0.5" layer="26" rot="MR90"/>
 <attribute name="VALUE" x="8.895" y="2.515" size="1.27" layer="28" rot="MR90"/>
@@
 <attribute name="VALUE" x="11.165" y="9.515" size="1.27" layer="27" rot="R180"/>
 </element>
-<element name="C17" library="rcl" package="C0603" value="1nF" x="28.3" y="2.82" smashed="yes" rot="MR90">
+<element name="C17" library="rcl" package="C0603" value="1000pF" x="28.3" y="2.82" smashed="yes" rot="MR90">
 <attribute name="NAME" x="28.935" y="2.185" size="0.5" layer="26" rot="MR90"/>
 <attribute name="VALUE" x="26.395" y="2.185" size="1.27" layer="28" rot="MR90"/>
@@
 <attribute name="VALUE" x="8.085" y="49.065" size="1.27" layer="27"/>
 </element>
-<element name="C8" library="rcl" package="C0603" value="1nF" x="2.42" y="31.37" smashed="yes" rot="MR180">
+<element name="C8" library="rcl" package="C0603" value="1000pF" x="2.42" y="31.37" smashed="yes" rot="MR180">
 <attribute name="NAME" x="2.035" y="30.735" size="0.5" layer="26" rot="MR180"/>
 <attribute name="VALUE" x="1.785" y="33.275" size="1.27" layer="28" rot="MR180"/>
@@
 <attribute name="VALUE" x="6.325" y="55.64" size="1.27" layer="27" rot="R90"/>
 </element>
-<element name="J1" library="RoboJackets-Connectors" package="2MM-2-V" value="2-PIN_2MM-V" x="81.18" y="68.7" smashed="yes" rot="R180">
-<attribute name="NAME" x="82.7425" y="68.95" size="0.5" layer="25" font="vector" ratio="10" rot="R180" align="bottom-center"/>
-<attribute name="PINS" value="2" x="81.18" y="68.7" size="1.778" layer="27" rot="R180" display="off"/>
-<attribute name="PIN_PITCH" value="2.0 mm" x="81.18" y="68.7" size="1.778" layer="27" rot="R180" display="off"/>
+<element name="J1" library="RoboJackets-Connectors" package="2MM-2-V" value="2-PIN_2MM-V" x="79.32" y="68.8" smashed="yes">
+<attribute name="NAME" x="77.7575" y="68.55" size="0.5" layer="25" font="vector" ratio="10" align="bottom-center"/>
+<attribute name="PINS" value="2" x="79.32" y="68.8" size="1.778" layer="27" display="off"/>
+<attribute name="PIN_PITCH" value="2.0 mm" x="79.32" y="68.8" size="1.778" layer="27" display="off"/>
 </element>
 <element name="JP1" library="adafruit" package="1X03" value="" x="80.47" y="3.88" smashed="yes" rot="R180">
@@
 </element>
 <element name="U$9" library="RoboJackets-Aesthetics" package="ROBOBUZZ_0.6X" value="" x="47.5" y="8.8125"/>
-<element name="R28" library="rcl" library_urn="urn:adsk.eagle:library:334" package="R0603" value="500" x="73" y="65.3125" rot="R180"/>
+<element name="R28" library="rcl" library_urn="urn:adsk.eagle:library:334" package="R0603" value="500" x="73" y="65.3125" smashed="yes" rot="R180">
+<attribute name="NAME" x="72.885" y="64.5525" size="0.5" layer="25" rot="R180"/>
+<attribute name="VALUE" x="73.635" y="67.2175" size="1.27" layer="27" rot="R180"/>
+</element>
 </elements>
 <signals>
@@
 <wire x1="12.22" y1="21.5925" x2="11" y2="22.8125" width="0.3" layer="16"/>
 <wire x1="11" y1="22.8125" x2="11" y2="24.75" width="0.3" layer="16"/>
-<wire x1="72.16" y1="67.3725" x2="71.5325" y2="68" width="0.3" layer="1"/>
-<wire x1="71.5325" y1="68" x2="71" y2="68" width="0.3" layer="1"/>
-<via x="71" y="68" extent="1-16" drill="0.35"/>
+<via x="71" y="67.9375" extent="1-16" drill="0.35"/>
+<wire x1="72.16" y1="67.3725" x2="71.565" y2="67.3725" width="0.3" layer="1"/>
+<wire x1="71.565" y1="67.3725" x2="71" y2="67.9375" width="0.3" layer="1"/>
 </signal>
 <signal name="N$2">
@@
 <wire x1="75" y1="58.5" x2="76" y2="59.5" width="0.3" layer="16"/>
 <wire x1="76" y1="59.5" x2="76" y2="64.5" width="0.3" layer="16"/>
-<wire x1="76" y1="64.5" x2="76.5" y2="65" width="0.3" layer="16"/>
-<wire x1="76.5" y1="65" x2="80" y2="65" width="0.3" layer="16"/>
-<wire x1="80" y1="65" x2="81.18" y2="66.18" width="0.3" layer="16"/>
 <contactref element="R28" pad="1"/>
-<wire x1="76" y1="64.5" x2="73.85" y2="65.3125" width="0" layer="19" extent="1-16"/>
+<wire x1="76" y1="64.5" x2="76.375" y2="64.875" width="0.3" layer="16"/>
+<via x="76.375" y="64.875" extent="1-16" drill="0.35"/>
+<wire x1="76.375" y1="64.875" x2="75.9375" y2="65.3125" width="0.3" layer="1"/>
+<wire x1="75.9375" y1="65.3125" x2="73.85" y2="65.3125" width="0.3" layer="1"/>
 </signal>
 <signal name="ESTOP_3V3">
@@
 <contactref element="R2" pad="1"/>
 <contactref element="Q1" pad="GATE"/>
-<wire x1="70.58" y1="69.15" x2="70.58" y2="71.24" width="0.3" layer="1"/>
-<wire x1="73.86" y1="68.64" x2="73.86" y2="67.3725" width="0.3" layer="1"/>
-<wire x1="73.35" y1="69.15" x2="73.86" y2="68.64" width="0.3" layer="1"/>
 <contactref element="J1" pad="1"/>
-<wire x1="73.86" y1="68.64" x2="81.18" y2="68.7" width="0" layer="19" extent="1-1"/>
-<wire x1="70.58" y1="69.15" x2="73.35" y2="69.15" width="0" layer="19" extent="1-1"/>
+<wire x1="79.32" y1="68.8" x2="78.02" y2="67.5" width="0.3" layer="1"/>
+<wire x1="78.02" y1="67.5" x2="77.5" y2="67.5" width="0.3" layer="1"/>
+<via x="77.5" y="67.5" extent="1-16" drill="0.35"/>
+<wire x1="77.5" y1="67.5" x2="74.875" y2="67.5" width="0.3" layer="16"/>
+<via x="74.875" y="67.5" extent="1-16" drill="0.35"/>
+<wire x1="74.875" y1="67.5" x2="74.7475" y2="67.3725" width="0.3" layer="1"/>
+<wire x1="73.86" y1="67.3725" x2="74.7475" y2="67.3725" width="0.3" layer="1"/>
+<wire x1="70.58" y1="68.92" x2="70.9625" y2="68.5375" width="0.3" layer="1"/>
+<wire x1="70.9625" y1="68.5375" x2="71.3257375" y2="68.5375" width="0.3" layer="1"/>
+<wire x1="72.8825" y1="68.35" x2="73.86" y2="67.3725" width="0.3" layer="1"/>
+<wire x1="71.3257375" y1="68.5375" x2="71.5132375" y2="68.35" width="0.3" layer="1"/>
+<wire x1="71.5132375" y1="68.35" x2="72.8825" y2="68.35" width="0.3" layer="1"/>
+<wire x1="70.58" y1="71.24" x2="70.58" y2="68.92" width="0.3" layer="1"/>
 </signal>
 <signal name="N$44">
@@
 <contactref element="J1" pad="2"/>
 <contactref element="R29" pad="2"/>
-<wire x1="72.1875" y1="69.15" x2="79.18" y2="68.7" width="0" layer="19" extent="1-1"/>
+<wire x1="81.32" y1="68.8" x2="80.12" y2="70" width="0.3" layer="1"/>
+<wire x1="80.12" y1="70" x2="78" y2="70" width="0.3" layer="1"/>
+<wire x1="78" y1="70" x2="77.5" y2="69.5" width="0.3" layer="1"/>
+<via x="77.5" y="69.5" extent="1-16" drill="0.35"/>
+<wire x1="77.5" y1="69.5" x2="77" y2="69" width="0.3" layer="16"/>
+<wire x1="77" y1="69" x2="74.5" y2="69" width="0.3" layer="16"/>
+<via x="74.5" y="69" extent="1-16" drill="0.35"/>
+<wire x1="74.5" y1="69" x2="74.35" y2="69.15" width="0.3" layer="1"/>
+<wire x1="74.35" y1="69.15" x2="72.1875" y2="69.15" width="0.3" layer="1"/>
 </signal>
 </signals>
