File: PCB/CarWarsPCB/CarWarsPCB/CarWarsPCBv_2.brd (EAGLE design)
At the start: 68.6 x 55.9 mm, 23 parts, among them J1 MAGJACK, Q1 220mA/50V/3.5Ω, Q2 220mA/50V/3.5Ω

Commit message: Updated design changes, under v2
Parts:
- removed J2: (no value), SparkFun-Connectors:USB-B-MICRO-SMD
Connections:
- removed net N$7: J2.D-, MBED.32
- removed net N$8: J2.D+, MBED.31
- net GND: no longer J2.GND, J2.SHIELD1, J2.SHIELD2, J2.SHIELD3
- net VCC: no longer J2.VBUS
Routing:
- net N$8: track 39.1 -> 0.00 mm, vias 2 -> 0
- net N$7: track 37.4 -> 0.00 mm, vias 2 -> 0
- net GND: track 52.6 -> 40.2 mm, vias 7 -> 4
- net VCC: track 97.5 -> 92.6 mm
- net DRIVE_PWM_12V: track 15.0 -> 11.9 mm
- net DRIVE_PWM_3V3: track 30.4 -> 29.9 mm
