File: neopixel_board/digikey_devices/SparkFun_Pro_Micro_v13a/SparkFun_Pro_Micro_v13a.sch (EAGLE design)
At the start: 35 parts, among them U1 UA7805CKCT, U2 MIC5219, U3 ATMEGA32U4, U4 UA7805CKCT, U5 UA7805CKCT, U6 UA7805CKCT, Y1 16MHz

Commit message: WIP cont
Need to connect connectors to neopixelstrips and ATMega pins. Look at resistor specs on voltage reg LEDs.
Parts:
- removed C7: (no value), rcl:C-USC0603
- removed ETH1: WIZ850IO, WIZ850io:WIZ850IO
- removed J1, J2, J3: (no value), SparkFun-Connectors:M04PTH
- removed PB1: PTS645PTS645_SMD1, Training_Board:PTS645PTS645_SMD1
- removed R1: (no value), rcl:R-US_R0603
- removed U1, U4, U5, U6: UA7805CKCT, Training_Board:UA7805CKCT
- added FRAME1: FRAME-LETTER, SparkFun-Aesthetics:FRAME-LETTER
- added JP1, JP2: FIDUCIALUFIDUCIAL, SparkFun:FIDUCIALUFIDUCIAL
- added JP6, JP7: M12PTH, SparkFun:M12PTH
- added SJ1: Closed for 5V Board, SparkFun:SOLDERJUMPERNC
- added U$1: LOGO-SFESK, SparkFun:LOGO-SFESK
- added U$11: LOGO-SFENEW, SparkFun:LOGO-SFENEW
- added U$3: OSHW-LOGOS, SparkFun:OSHW-LOGOS
- R2: value (none) -> 10K; device rcl:R-US_R0603 -> SparkFun:RESISTOR0603-RES
Connections:
- removed net INTN: ETH1.6
- removed net N$10: C7.1, ETH1.8, ETH1.9, R2.1
- removed net N$9: D2.A, F1.2
- removed net RST: PB1.1, R1.2, U3.!RESET
- removed net SCLK: ETH1.4
- removed net SCNN: ETH1.5
- removed net VCC_ATMEG: U3.AVCC@24, U3.AVCC@44, U3.VCC@14, U3.VCC@34
- new net N$3: D2.A, F1.2, SJ1.1
- new net RESET: JP6.3, R2.1, U3.!RESET
- net A0: now also JP6.8
- net A1: now also JP6.7
- net A2: now also JP6.6
- net A3: now also JP6.5
- net D10: now also JP6.12
- net D2: now also JP7.8
- net D3: now also JP7.7
- net D4: now also JP7.6
- net D5: now also JP7.5
- net D6: now also JP7.4
- net D7: now also JP7.3
- net D8: now also JP7.2
- net D9: now also JP7.1
- net GND: now also JP6.2, JP7.10, JP7.9; no longer C7.2, ETH1.1, ETH1.2, ETH1.7, PB1.2
- net MISO: now also JP6.10
- net MOSI: now also JP6.11; no longer ETH1.3
- net RAW: now also JP6.1
- net RXI: now also JP7.11
- net SCK: now also JP6.9
- net TXO: now also JP7.12
- net VCC: now also JP6.4, R2.2, SJ1.2, U3.AVCC@24, U3.AVCC@44, U3.VCC@14, U3.VCC@34; no longer R1.1
Other:
- note added: "Added fuse and diode protection"
- note added: "Added two small squares of tRestrict to keep the ground plane away from the sides of IC legs"
- note added: "Arduino Pro Mini Design by Spark Fun Electronics"
- note added: "Change to 500mA regulator"
- note added: "Changed LEDs to be tied to VCC"
- note added: "Changes on v1.1:"
- note added: "Changes on v1.2:"
- note added: "Changes on v1.3:"
- note added: "Corrected silk on D14"
- note added: "Open for 3.3V Board"
- note added: "Original Arduino Mini Design by Team Arduino"
- note added: "Pro Micro Design by Spark Fun Electronics"
- note added: "Renamed SS net to D14 (from D17)"
- note added: "Routed directly inward or outward from each leg on the IC"
- note added: "Updated QFN package on 32U4 to be 1:1"
- note added: "Updated package on USB micro B (2 new pads)"
- note added: "Updated symbol of 32U4 in schematic (switched MISO and SS placement)"
- note added: "v13"
- note removed: "Reset PB"
- moved on the sheet: C1, C10, C13, C19, C2, C3, C4, C5, C6, D1, D2, D3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
