File: lidar-breakout/Archive/LIDAR_Breakout.brd (EAGLE design)
At the start: 36.5 x 88 mm, 83 parts

Commit message: Routing Updates, Design Review Updates, Cleanup
Parts:
- removed C11: 0.1 uF, resistor:C0603
- removed C24, C25: 10 uF, rcl:E2-5
- removed F4, F5, F6, F7, F8, F9: 200mA, RoboJackets-Fuses:F0603
- removed LD4: GREEN, led:CHIP-LED0603
- removed P2: (no value), adafruit:DCJACK_2MM_PTH
- removed R5, R6: 4.7 kΩ, rcl:R0603
- removed USB1: (no value), microbuilder:4UCONN_20329
- added 5V-REGULATED: (no value), 0436500200:MOLEX_0436500200
- added C1, C2: 10 uF, EEE-1CA100SR:CAPAE430X550N
- added D3: (no value), RoboJackets-Diodes:DO-214AC
- added I2C_LED: YELLOW, led:CHIP-LED0603
- added Q2: (no value), RoboJackets-Discrete:SOT-23-3
- added USB: (no value), 47589-0001:MOLEX_47589-0001
- moved U$3 70.8 mm to (30.2, 1.20)
- moved R3 22.2 mm to (27.0, 28.7), turned to 270 degrees
- moved PB2 18.8 mm to (1.20, 72.8), turned to 270 degrees
- moved C10 9.91 mm to (26.5, 72.0), flipped to the top, turned to 270 degrees
- moved TP4 8.76 mm to (14.4, 39.0)
- moved R15 8.08 mm to (4.81, 31.7), flipped to the top, turned to 90 degrees
- moved H1 8.05 mm to (28.9, 79.0)
- moved LD7 8.02 mm to (16.1, 77.9), turned to 0 degrees
- moved R16 6.77 mm to (7.91, 35.6), flipped to the top, turned to 90 degrees
- moved R7 5.90 mm to (15.8, 74.7), flipped to the top, turned to 180 degrees
- moved TP3 5.60 mm to (21.3, 67.0)
- moved R8 4.61 mm to (30.0, 74.0), flipped to the top, turned to 90 degrees
- moved F3 4.52 mm to (18.1, 45.2), turned to 180 degrees
- moved R10 4.52 mm to (30.1, 45.0), flipped to the top, turned to 90 degrees
- moved R9 4.22 mm to (30.1, 59.9), flipped to the top, turned to 90 degrees
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Connections:
- net DATA_N renamed USB_N
- net DATA_P renamed USB_P
- removed net 5VREG: C22.1, C25.+, F2.2, F3.2, P2.PWR, R2.2, TP2.TP, VR1.4
- removed net I2C_ACT: MC1.26, R3.2
- removed net VCC_LDR0: F4.1, H1.P$3
- removed net VCC_LDR1: F5.1, H2.P$3
- removed net VCC_LDR2: F6.1, H3.P$3
- removed net VCC_LDR3: F7.1, H4.P$3
- removed net VCC_LDR4: F8.1, H5.P$3
- removed net VCC_LDR5: F9.1, H6.P$3
- new net I2C_ACTIVITY: MC1.29, R3.1
- new net N$14: R16.2, USB.2
- new net N$9: 5V-REGULATED.2, Q2.2
- new net VOUT: C2.1, C22.1, F2.2, F3.2, Q2.3, R2.2, TP2.TP, VR1.4
- net GND: now also 5V-REGULATED.1, C1.2, C2.2, I2C_LED.C, Q2.1, USB.5, USB.P$1, USB.P$2, USB.P$3, USB.P$4, USB.P$5, USB.P$6; no longer C11.2, C24.-, C25.-, LD4.C, P2.GND, P2.GNDBREAK, USB1.BASE@1, USB1.BASE@2, USB1.GND, USB1.SPRT@1, USB1.SPRT@2, USB1.SPRT@3, USB1.SPRT@4
- net N$1: now also USB.1; no longer USB1.VBUS
- net N$2: now also D3.A, P1.2; no longer LD4.A, R3.1
- net N$23: now also USB.3; no longer USB1.D+
- net N$8: now also I2C_LED.A, R3.2; no longer R16.2, USB1.D-
- net SCL_LIDAR: no longer R6.2
- net SDA_LIDAR: no longer R5.2
- net UVCC: now also D3.C; no longer P1.2
- net VCC_1: now also H1.P$3, H2.P$3, H3.P$3, H4.P$3, H5.P$3, H6.P$3; no longer C11.1, F4.2, F5.2, F6.2, F7.2, F8.2, F9.2, R5.1, R6.1
- net VIN: now also C1.1; no longer C24.+
Routing:
- net VOUT: track 0.00 -> 76.0 mm, vias 0 -> 4
- net 5VREG: track 68.9 -> 0.00 mm, vias 4 -> 0
- net I2C_ACT: track 58.1 -> 0.00 mm, vias 2 -> 0
- net GND: track 168.8 -> 110.9 mm, vias 49 -> 51
- net USB_N: track 40.2 -> 0.00 mm, vias 1 -> 0
- net USB_P: track 40.3 -> 0.58 mm, vias 1 -> 0
- net I2C_ACTIVITY: track 0.00 -> 20.9 mm
- net VCC_1: track 102.2 -> 121.4 mm, vias 1 -> 4
- net RST_MC: track 105.5 -> 87.9 mm
- net RST_ETH: track 86.8 -> 69.7 mm, vias 4 -> 2
- net SDA_LIDAR: track 134.4 -> 118.1 mm
- net MISO_ETH: track 43.9 -> 31.3 mm, vias 2 -> 1
- net SCL_LIDAR: track 138.8 -> 128.2 mm
- net UVCC: track 15.5 -> 8.57 mm
- net INTN_ETH: track 7.86 -> 14.6 mm, vias 1 -> 2
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Other:
- board size 36.5 x 88 mm -> 36.5 x 80 mm
- board text added: "SCL"
- board text added: "SDA"
- board text removed: "5VDC_REG"
- board text removed: "I2C_ACT"
