File: lidar-breakout/V2/LIDAR_Breakout_V2.sch (EAGLE design)
At the start: 81 parts, among them P1 MOLEX 0436500200, X1 TSX-3225 16.0000MF18X-AC0

Commit message: Switched LED directions, Fixed I2C pulled resistor
Parts:
- added IO1: PCA9555DB, micro-philips:PCA9555DB
- added LD13, LD14, LD15, LD16, LD17, LD5, LD6: RED, RoboJackets-LEDs:LED-SMD-RED
- added LD18, LD19: GREEN, led:LEDCHIP-LED0603
- added R17, R18, R19: 1 kΩ, rcl:R-US_R0603
- added R24: 2NBS16-8, resistor-bourns:2NBS16-8
- added U1: PCA9548ADBR, PCA9548ADBR:PCA9548ADBR
Connections:
- new net COMM_ERR: R17.1
- new net LDR2_ERR: LD13.A, R24.13
- new net LDR6_ERR: LD14.A, LD15.A, LD16.A, LD17.A, LD6.A, R24.10, R24.11, R24.12, R24.14, R24.9
- new net N$10: LD15.K
- new net N$11: LD18.A, R18.1
- new net N$12: LD19.A, R19.1
- new net N$16: LD16.K
- new net N$18: LD14.K
- new net N$19: LD13.K
- new net N$20: IO1.I/O1.0, R24.1
- new net N$21: IO1.I/O1.1, R24.2
- new net N$22: IO1.I/O1.2, R24.3
- new net N$24: IO1.I/O1.3, R24.4
- new net N$25: IO1.I/O1.4, R24.5
- new net N$26: IO1.I/O1.5, R24.6
- new net N$27: IO1.I/O1.6, R24.7
- new net N$28: IO1.I/O1.7, R24.8
- new net N$9: LD5.A, R17.2
- net GND: now also IO1.VSS, LD17.K, LD18.C, LD19.C, LD5.K, LD6.K
- net SCL: now also IO1.SCL
- net SDA: now also IO1.SDA
- net VCC_1: now also R19.2
- net VCC_2: now also IO1.VDD, R18.2
Other:
- note added: "COMM ERROR"
- note added: "LDR1 ERROR"
- note added: "LDR2 ERROR"
- note added: "LDR3 ERROR"
- note added: "LDR4 ERROR"
- note added: "LDR5 ERROR"
- note added: "LDR6 ERROR"
- note added: "LIDAR POWER OK"
- note added: "Lidar Error LEDs"
- note added: "MC POWER OK"
- moved on the sheet: C22, D2, F2, F3
