File: estop_daugherboard/EVGP Daugherboard.sch (EAGLE design)
At the start: 24 parts, among them J2 AVR_SPI_PROG_3X2PTH, J3 UX60-MB-5S8, U1 ATMEGA32U4-AU, X1 TSX-3225 16.0000MF18X-AC0

Commit message: estop daugherboard stuff
Parts:
- added C11, C12: big, resistor:C-USC0603
- added F1: 0.2A, adafruit:PTCFUSE-1206
- added R2: 10kΩ, rcl:R-US_R0603
- added U2, U3: (no value), DownloadedParts:BSS84DW-7-F
- C9: value (none) -> big; device rcl:CPOL-USE2.5-7 -> resistor:C-USC0603
Connections:
- net STACK_LED1: now also U2.G1
Changed lines of the file:
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@@
 <part name="GND10" library="SparkFun-PowerSymbols" deviceset="GND" device=""/>
 <part name="R14" library="rcl" library_urn="urn:adsk.eagle:library:334" deviceset="R-US_" device="R0603" package3d_urn="urn:adsk.eagle:package:23555/2" value="330Ω"/>
-<part name="C9" library="rcl" library_urn="urn:adsk.eagle:library:334" deviceset="CPOL-US" device="E2.5-7" package3d_urn="urn:adsk.eagle:package:23345/1"/>
+<part name="R2" library="rcl" library_urn="urn:adsk.eagle:library:334" deviceset="R-US_" device="R0603" package3d_urn="urn:adsk.eagle:package:23555/2" value="10kΩ"/>
+<part name="C9" library="resistor" library_urn="urn:adsk.eagle:library:348" deviceset="C-US" device="C0603" package3d_urn="urn:adsk.eagle:package:23616/2" value="big"/>
+<part name="C11" library="resistor" library_urn="urn:adsk.eagle:library:348" deviceset="C-US" device="C0603" package3d_urn="urn:adsk.eagle:package:23616/2" value="big"/>
+<part name="C12" library="resistor" library_urn="urn:adsk.eagle:library:348" deviceset="C-US" device="C0603" package3d_urn="urn:adsk.eagle:package:23616/2" value="big"/>
+<part name="U2" library="DownloadedParts" deviceset="BSS84DW-7-F" device=""/>
+<part name="U3" library="DownloadedParts" deviceset="BSS84DW-7-F" device=""/>
+<part name="P+1" library="supply1" library_urn="urn:adsk.eagle:library:371" deviceset="+24V" device=""/>
+<part name="F1" library="adafruit" library_urn="urn:adsk.eagle:library:420" deviceset="PTCFUSE" device="-1206" package3d_urn="urn:adsk.eagle:package:6240569/1" value="0.2A"/>
 </parts>
 <sheets>
@@
 <text x="170.18" y="96.52" size="5.08" layer="97">Stack Light</text>
 <wire x1="165.1" y1="106.68" x2="165.1" y2="10.16" width="0.1524" layer="97" style="shortdash"/>
-<wire x1="165.1" y1="10.16" x2="228.6" y2="10.16" width="0.1524" layer="97" style="shortdash"/>
-<wire x1="228.6" y1="10.16" x2="228.6" y2="106.68" width="0.1524" layer="97" style="shortdash"/>
-<wire x1="228.6" y1="106.68" x2="165.1" y2="106.68" width="0.1524" layer="97" style="shortdash"/>
+<wire x1="165.1" y1="10.16" x2="322.58" y2="10.16" width="0.1524" layer="97" style="shortdash"/>
+<wire x1="322.58" y1="10.16" x2="322.58" y2="106.68" width="0.1524" layer="97" style="shortdash"/>
+<wire x1="322.58" y1="106.68" x2="165.1" y2="106.68" width="0.1524" layer="97" style="shortdash"/>
 </plain>
 <instances>
@@
 <attribute name="VALUE" x="145.542" y="120.65" size="1.778" layer="96" rot="R90"/>
 </instance>
-<instance part="C9" gate="G$1" x="185.42" y="66.04" smashed="yes">
-<attribute name="NAME" x="186.436" y="66.675" size="1.778" layer="95"/>
-<attribute name="VALUE" x="186.436" y="61.849" size="1.778" layer="96"/>
+<instance part="R2" gate="G$1" x="182.88" y="48.26" smashed="yes" rot="R90">
+<attribute name="NAME" x="181.3814" y="44.45" size="1.778" layer="95" rot="R90"/>
+<attribute name="VALUE" x="186.182" y="44.45" size="1.778" layer="96" rot="R90"/>
+</instance>
+<instance part="C9" gate="G$1" x="274.32" y="81.28" smashed="yes">
+<attribute name="NAME" x="275.336" y="81.915" size="1.778" layer="95"/>
+<attribute name="VALUE" x="275.336" y="77.089" size="1.778" layer="96"/>
+</instance>
+<instance part="C11" gate="G$1" x="193.04" y="27.94" smashed="yes">
+<attribute name="NAME" x="194.056" y="28.575" size="1.778" layer="95"/>
+<attribute name="VALUE" x="194.056" y="23.749" size="1.778" layer="96"/>
+</instance>
+<instance part="C12" gate="G$1" x="177.8" y="27.94" smashed="yes">
+<attribute name="NAME" x="178.816" y="28.575" size="1.778" layer="95"/>
+<attribute name="VALUE" x="178.816" y="23.749" size="1.778" layer="96"/>
+</instance>
+<instance part="U2" gate="A" x="264.16" y="73.66" smashed="yes" rot="R180">
+<attribute name="NAME" x="253.6444" y="64.5414" size="2.0828" layer="95" ratio="6" rot="SR180"/>
+<attribute name="VALUE" x="254.2794" y="67.0814" size="2.0828" layer="96" ratio="6" rot="SR180"/>
+</instance>
+<instance part="U3" gate="A" x="264.16" y="48.26" smashed="yes" rot="R180">
+<attribute name="NAME" x="253.6444" y="39.1414" size="2.0828" layer="95" ratio="6" rot="SR180"/>
+<attribute name="VALUE" x="254.2794" y="41.6814" size="2.0828" layer="96" ratio="6" rot="SR180"/>
+</instance>
+<instance part="P+1" gate="1" x="220.98" y="88.9" smashed="yes" rot="R180">
+<attribute name="VALUE" x="223.52" y="93.98" size="1.778" layer="96" rot="R270"/>
+</instance>
+<instance part="F1" gate="G$1" x="257.302" y="134.62" smashed="yes">
+<attribute name="VALUE" x="252.222" y="134.112" size="1.778" layer="96"/>
+<attribute name="NAME" x="259.08" y="134.112" size="1.778" layer="95"/>
 </instance>
 </instances>
@@
 <label x="121.92" y="58.42" size="1.27" layer="95" font="vector" xref="yes"/>
 </segment>
+<segment>
+<pinref part="U2" gate="A" pin="G1"/>
+<wire x1="236.22" y1="76.2" x2="187.96" y2="76.2" width="0.1524" layer="91"/>
+<label x="187.96" y="76.2" size="1.27" layer="95" rot="R180" xref="yes"/>
+</segment>
 </net>
 <net name="STACK_LED2" class="0">
@@
 packages will not be understood (or retained) with this version.
 </note>
-<note version="8.4" severity="warning">
-Since Version 8.4, EAGLE supports properties for SPICE simulation.
-Probes in schematics and SPICE mapping objects found in parts and library devices
-will not be understood with this version. Update EAGLE to the latest version
-for full support of SPICE simulation.
-</note>
 </compatibility>
