File: new-cari/manual-rc/manual-rc.sch (EAGLE design)
At the start: 22 parts, among them J5 1734510-1, X1 TSX-3225 16.0000MF18X-AC0

Commit message: Manual RC Board WIP v2
Parts:
- removed PB3: PTS645PTS645_SMD1, Training_Board:PTS645PTS645_SMD1
- added PB1: ATMEGA_RESET, RoboJackets-Switches:PB_RA
- PB2: value PTS645PTS645_SMD1 -> ATMEGA_RESET; device Training_Board:PTS645PTS645_SMD1 -> RoboJackets-Switches:PB_RA
Connections:
- net N$6 renamed D2_N
- net N$9 renamed D2_P
- new net INTN: MC1.PD3(INT3/TXD1), U$2.INTN
- net GND: now also PB1.2; no longer PB3.2
- net RST_MC: now also PB1.1; no longer PB3.1
Changed lines of the file:
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@@
 <part name="U$1" library="manual-rc" deviceset="HK-GT2B" device="" package3d_urn="urn:adsk.eagle:package:14970250/1"/>
 <part name="P+3" library="supply1" library_urn="urn:adsk.eagle:library:371" deviceset="+5V" device=""/>
-<part name="U$2" library="ethernet_poe" deviceset="ETH-POE" device="" package3d_urn="urn:adsk.eagle:package:14970482/1"/>
 <part name="SUPPLY7" library="supply2" library_urn="urn:adsk.eagle:library:372" deviceset="GND" device=""/>
 <part name="P+4" library="supply1" library_urn="urn:adsk.eagle:library:371" deviceset="+5V" device=""/>
@@
 <part name="R2" library="rcl" library_urn="urn:adsk.eagle:library:334" deviceset="R-US_" device="R0603" package3d_urn="urn:adsk.eagle:package:23555/3" value="10 kΩ"/>
 <part name="P+5" library="supply1" library_urn="urn:adsk.eagle:library:371" deviceset="+5V" device=""/>
-<part name="PB2" library="Training_Board" deviceset="PTS645" device="PTS645_SMD1"/>
-<part name="PB3" library="Training_Board" deviceset="PTS645" device="PTS645_SMD1"/>
 <part name="FRAME1" library="RoboJackets-Frames" deviceset="FRAME_A_L" device=""/>
 <part name="J5" library="1734510-1" deviceset="1734510-1" device=""/>
@@
 <part name="D1" library="SparkFun" deviceset="DIODE" device="SOD"/>
 <part name="SUPPLY6" library="supply2" library_urn="urn:adsk.eagle:library:372" deviceset="GND" device=""/>
+<part name="U$2" library="ethernet_poe" deviceset="ETH-POE" device="" package3d_urn="urn:adsk.eagle:package:14970482/1"/>
+<part name="PB1" library="RoboJackets-Switches" deviceset="PB_RA" device="" value="ATMEGA_RESET"/>
+<part name="PB2" library="RoboJackets-Switches" deviceset="PB_RA" device="" value="ATMEGA_RESET"/>
 </parts>
 <sheets>
@@
 <attribute name="VALUE" x="129.54" y="167.64" size="1.778" layer="96" rot="R90"/>
 </instance>
-<instance part="U$2" gate="POE-DEMO" x="228.6" y="86.36" smashed="yes">
-<attribute name="NAME" x="218.44" y="96.52" size="1.778" layer="95"/>
-<attribute name="VALUE" x="218.44" y="68.58" size="1.778" layer="96"/>
-</instance>
 <instance part="SUPPLY7" gate="GND" x="205.74" y="91.44" smashed="yes">
 <attribute name="VALUE" x="208.915" y="90.805" size="1.778" layer="96"/>
@@
 <instance part="P+5" gate="1" x="215.9" y="127" smashed="yes">
 <attribute name="VALUE" x="213.36" y="121.92" size="1.778" layer="96" rot="R90"/>
-</instance>
-<instance part="PB2" gate="G$1" x="226.06" y="111.76" smashed="yes">
-<attribute name="NAME" x="220.98" y="115.57" size="1.778" layer="95" font="vector"/>
-<attribute name="VALUE" x="226.06" y="110.49" size="2.54" layer="96" font="vector" ratio="15" align="top-center" display="off"/>
-</instance>
-<instance part="PB3" gate="G$1" x="226.06" y="142.24" smashed="yes">
-<attribute name="NAME" x="220.98" y="146.05" size="1.778" layer="95" font="vector"/>
-<attribute name="VALUE" x="226.06" y="140.97" size="2.54" layer="96" font="vector" ratio="15" align="top-center" display="off"/>
 </instance>
 <instance part="FRAME1" gate="G$1" x="0" y="0" smashed="yes"/>
@@
 <instance part="SUPPLY6" gate="GND" x="132.08" y="162.56" smashed="yes">
 <attribute name="VALUE" x="135.255" y="161.925" size="1.778" layer="96"/>
+</instance>
+<instance part="U$2" gate="POE-DEMO" x="228.6" y="86.36" smashed="yes">
+<attribute name="NAME" x="218.44" y="96.52" size="1.778" layer="95"/>
+<attribute name="VALUE" x="218.44" y="68.58" size="1.778" layer="96"/>
+</instance>
+<instance part="PB1" gate="G$1" x="226.06" y="142.24" smashed="yes">
+<attribute name="NAME" x="223.52" y="146.05" size="1.778" layer="95" font="vector"/>
+<attribute name="VALUE" x="226.06" y="140.97" size="1.778" layer="96" font="vector" align="top-center"/>
+</instance>
+<instance part="PB2" gate="G$1" x="226.06" y="111.76" smashed="yes">
+<attribute name="NAME" x="223.52" y="115.57" size="1.778" layer="95" font="vector"/>
+<attribute name="VALUE" x="226.06" y="110.49" size="1.778" layer="96" font="vector" align="top-center"/>
 </instance>
 </instances>
@@
 <segment>
 <pinref part="P+4" gate="1" pin="+5V"/>
+<wire x1="205.74" y1="83.82" x2="213.36" y2="83.82" width="0.1524" layer="91"/>
 <pinref part="U$2" gate="POE-DEMO" pin="+5V"/>
-<wire x1="205.74" y1="83.82" x2="213.36" y2="83.82" width="0.1524" layer="91"/>
 </segment>
 </net>
@@
 <wire x1="238.76" y1="152.4" x2="238.76" y2="142.24" width="0.1524" layer="91"/>
 <junction x="238.76" y="142.24"/>
-<pinref part="PB3" gate="G$1" pin="2"/>
-</segment>
-<segment>
-<pinref part="U$2" gate="POE-DEMO" pin="GND"/>
+<pinref part="PB1" gate="G$1" pin="2"/>
+</segment>
+<segment>
 <pinref part="SUPPLY7" gate="GND" pin="GND"/>
 <wire x1="213.36" y1="93.98" x2="205.74" y2="93.98" width="0.1524" layer="91"/>
+<pinref part="U$2" gate="POE-DEMO" pin="GND"/>
 </segment>
 <segment>
@@
 <junction x="215.9" y="142.24"/>
 <label x="210.82" y="142.24" size="1.016" layer="95" rot="MR0" xref="yes"/>
-<pinref part="PB3" gate="G$1" pin="1"/>
+<pinref part="PB1" gate="G$1" pin="1"/>
 <junction x="220.98" y="142.24"/>
 </segment>
@@
 <segment>
 <pinref part="C8" gate="G$1" pin="1"/>
-<wire x1="88.9" y1="160.02" x2="88.9" y2="162.56" width="0.1524" layer="91"/>
+<wire x1="88.9" y1="160.02" x2="86.36" y2="162.56" width="0.1524" layer="91"/>
 <pinref part="X1" gate="G$1" pin="1"/>
-<wire x1="88.9" y1="162.56" x2="93.98" y2="162.56" width="0.1524" layer="91"/>
-<wire x1="88.9" y1="162.56" x2="83.82" y2="162.56" width="0.1524" layer="91"/>
-<junction x="88.9" y="162.56"/>
+<wire x1="86.36" y1="162.56" x2="93.98" y2="162.56" width="0.1524" layer="91"/>
+<wire x1="86.36" y1="162.56" x2="83.82" y2="162.56" width="0.1524" layer="91"/>
+<junction x="86.36" y="162.56"/>
 <label x="83.82" y="162.56" size="1.016" layer="95" rot="MR0" xref="yes"/>
 </segment>
@@
 </segment>
 <segment>
-<pinref part="U$2" gate="POE-DEMO" pin="MISO"/>
 <wire x1="243.84" y1="83.82" x2="248.92" y2="83.82" width="0.1524" layer="91"/>
 <label x="248.92" y="83.82" size="1.016" layer="95" xref="yes"/>
+<pinref part="U$2" gate="POE-DEMO" pin="MISO"/>
 </segment>
 </net>
@@
 </segment>
 <segment>
-<pinref part="U$2" gate="POE-DEMO" pin="MOSI"/>
 <wire x1="243.84" y1="78.74" x2="248.92" y2="78.74" width="0.1524" layer="91"/>
 <label x="248.92" y="78.74" size="1.016" layer="95" xref="yes"/>
+<pinref part="U$2" gate="POE-DEMO" pin="MOSI"/>
 </segment>
 </net>
@@
 </segment>
 <segment>
-<pinref part="U$2" gate="POE-DEMO" pin="SCLK"/>
 <wire x1="243.84" y1="88.9" x2="248.92" y2="88.9" width="0.1524" layer="91"/>
 <label x="248.92" y="88.9" size="1.016" layer="95" xref="yes"/>
+<pinref part="U$2" gate="POE-DEMO" pin="SCLK"/>
 </segment>
 </net>
@@
 </segment>
 <segment>
-<pinref part="U$2" gate="POE-DEMO" pin="SCSN"/>
 <wire x1="243.84" y1="93.98" x2="248.92" y2="93.98" width="0.1524" layer="91"/>
 <label x="248.92" y="93.98" size="1.016" layer="95" xref="yes"/>
+<pinref part="U$2" gate="POE-DEMO" pin="SCSN"/>
 </segment>
 </net>
@@
 <wire x1="226.06" y1="121.92" x2="220.98" y2="121.92" width="0.1524" layer="91"/>
 <wire x1="220.98" y1="121.92" x2="220.98" y2="111.76" width="0.1524" layer="91"/>
-<wire x1="220.98" y1="111.76" x2="215.9" y2="111.76" width="0.1524" layer="91"/>
+<pinref part="PB2" gate="G$1" pin="1"/>
 <pinref part="R2" gate="G$1" pin="1"/>
 <wire x1="215.9" y1="111.76" x2="210.82" y2="111.76" width="0.1524" layer="91"/>
+<label x="210.82" y="111.76" size="1.016" layer="95" rot="R180" xref="yes"/>
+<wire x1="215.9" y1="111.76" x2="220.98" y2="111.76" width="0.1524" layer="91"/>
 <junction x="215.9" y="111.76"/>
-<label x="210.82" y="111.76" size="1.016" layer="95" rot="R180" xref="yes"/>
-<pinref part="PB2" gate="G$1" pin="1"/>
 <junction x="220.98" y="111.76"/>
 </segment>
 <segment>
-<pinref part="U$2" gate="POE-DEMO" pin="RSTN"/>
 <wire x1="213.36" y1="78.74" x2="208.28" y2="78.74" width="0.1524" layer="91"/>
 <label x="208.28" y="78.74" size="1.016" layer="95" rot="MR0" xref="yes"/>
+<pinref part="U$2" gate="POE-DEMO" pin="RSTN"/>
 </segment>
 <segment>
@@
 </segment>
 </net>
-<net name="N$6" class="0">
+<net name="D2_N" class="2">
 <segment>
 <wire x1="223.52" y1="185.42" x2="208.28" y2="185.42" width="0.1524" layer="91"/>
@@
 </segment>
 </net>
-<net name="N$9" class="0">
+<net name="D2_P" class="2">
 <segment>
 <wire x1="223.52" y1="182.88" x2="213.36" y2="182.88" width="0.1524" layer="91"/>
@@
 </segment>
 </net>
+<net name="INTN" class="0">
+<segment>
+<pinref part="U$2" gate="POE-DEMO" pin="INTN"/>
+<wire x1="243.84" y1="73.66" x2="248.92" y2="73.66" width="0.1524" layer="91"/>
+<label x="248.92" y="73.66" size="1.016" layer="95" xref="yes"/>
+</segment>
+<segment>
+<pinref part="MC1" gate="G$1" pin="PD3(INT3/TXD1)"/>
+<wire x1="182.88" y1="73.66" x2="185.42" y2="73.66" width="0.1524" layer="91"/>
+<label x="185.42" y="73.66" size="1.016" layer="95" xref="yes"/>
+</segment>
+</net>
