File: distributed-vision/DistributedVisionSchematicPage1_33.sch (EAGLE design)
At the start: 114 parts, among them J1 RASPBERRRY_COMPUTE_CM3, J2 RASPBERRRY_COMPUTE_CM3, J3 XS10, J4 10029449-111RLF, J5 10029449-111RLF, Q1 AP2331SA-7, Q2 BSS127, Q3 BSS127, Q4 BJT-NPN_, U1 TPS70625DBVR, U2 LM26420XMH, U3 TPD13S523, U4 ESD224, X1 JST-XH-02-PIN-LONG-PAD

Commit message: Finished Page 3, Re-working Page 1
Parts:
- removed C102, C103, C69, C70, C71, C72, C76, C77, C78, C79, C80, C81, C82, C83, C84, C85, C88, C91: (no value), rcl:C-USC0603
- removed C52, C58: 10n, rcl:C-USC0603
- removed DQ1, DQ2, DQ6: GREEN, RoboJackets-LEDs:LED-GREEN0603
- removed F1: (no value), RoboJackets-Fuses:PTCFUSE-1812
- removed J1, J2: RASPBERRRY_COMPUTE_CM3, distributed-vision:RASPBERRRY_COMPUTE_CM3
- removed J3: XS10, distributed-vision:XS10
- removed J4, J5: 10029449-111RLF, distributed-vision:10029449-111RLF
- removed L2, L3: (no value), RoboJackets-Inductors:INDUCTOR_0805
- removed Q2, Q3: BSS127, RoboJackets-Discrete:BSS127
- removed Q4: BJT-NPN_, RoboJackets-Discrete:BJT-NPN_
- removed R10: 31k6, rcl:R-US_R0603
- removed R11: 12k7, rcl:R-US_R0603
- removed R12, R25, R44: 470r, rcl:R-US_R0603
- removed R13, R15, R17, R2, R45, R5, R6, R7: (no value), rcl:R-US_R0603
- removed R14: 10k, rcl:R-US_R0603
- removed R16, R20, R21, R22, R49, R50: 4k7, rcl:R-US_R0603
- removed R23, R24, R4: 100k, rcl:R-US_R0603
- removed R55, R8, R9: 47k, rcl:R-US_R0603
- removed S2: 34EWMSP12M6RT, RoboJackets-Switches:34EWMSP12M6RT
- removed U3: TPD13S523, distributed-vision:TPD13S523
- removed U4: ESD224, distributed-vision:ESD224
- removed VD4: 60V, RoboJackets-Diodes:DFLS160-7
- removed X1: JST-XH-02-PIN-LONG-PAD, RoboJackets-Connectors:JST-XH-02-PIN-LONG-PAD
- added C14, C20, C42, C43, C44, C49, C50: (no value), rcl:C-USC0603
- added D1: 75V, RoboJackets-Diodes:1N4148WX
- C26, C27, C28, C29: value 22u -> (none); device rcl:C-USC0805 -> rcl:C-USC0603
- C45, C46: value 100n -> (none)
- R1: value 47k -> (none)
Connections:
- removed net CAM0_IO0: J2A.GPIO44, J4.11, R24.2
- removed net CAM0_IO1: J2A.GPIO39, J4.12
- removed net CAM0_SCL: J2A.GPIO1, J4.13, R16.2
- removed net CAM0_SDA: J2A.GPIO0, J4.14, R20.2
- removed net CAM1_IO0: J2A.GPIO45, J5.11, R23.2
- removed net CAM1_IO1: J2A.GPIO37, J5.12
- removed net CAM1_SCL: J2A.GPIO29, J5.13, R22.2
- removed net CAM1_SDA: J2A.GPIO28, J5.14, R21.2
- removed net EMMC_DISABLE_N: J1A.!EMMC_DISABLE, Q2.D
- removed net EMMC_EN_N_1V8: J1B.EMMC_EN_N_1V8, Q3.G, R4.1
- removed net FB1: R10.1
- removed net FB2: C28.1, C29.1, L2.2, R11.1
- removed net GPIO02: J2A.GPIO2, J3.GPIO02, R49.1
- removed net GPIO03: J2A.GPIO3, J3.GPIO03, R50.1
- removed net GPIO04: J2A.GPIO4, J3.GPIO04
- removed net GPIO05: J2A.GPIO5, J3.GPIO05
- removed net GPIO06: J2A.GPIO6, J3.GPIO06
- removed net GPIO07: J2A.GPIO7, J3.GPIO07
- removed net GPIO08: J2A.GPIO8, J3.GPIO08
- removed net GPIO12: J2A.GPIO12, J3.GPIO12
- removed net GPIO13: J2A.GPIO13, J3.GPIO13
- removed net GPIO14: J2A.GPIO14, J3.GPIO14
- removed net GPIO15: J2A.GPIO15, J3.GPIO15
- removed net GPIO16: J2A.GPIO16, J3.GPIO16
- removed net GPIO18: J2A.GPIO18, J3.GPIO18
- removed net GPIO19: J2A.GPIO19, J3.GPIO19
- removed net GPIO20: J2A.GPIO20, J3.GPIO20
- removed net GPIO21: J2A.GPIO21, J3.GPIO21
- removed net GPIO23: J2A.GPIO23, J3.GPIO23
- removed net GPIO24: J2A.GPIO24, J3.GPIO24
- removed net GPIO25: J2A.GPIO25, J3.GPIO25
- removed net GPIO38_RESET: J2A.GPIO38
- removed net N$1: R10.2, R13.2, U2.FB1
- removed net N$10: J2A.GPIO17, J3.GPIO17
- removed net N$11: J2A.GPIO26, J3.GPIO26
- removed net N$12: J2A.CAM1_CP, J5.9
- removed net N$13: J2A.CAM1_CN, J5.8
- removed net N$14: J2A.CAM1_DP1, J5.6
- removed net N$15: J2A.CAM1_DN1, J5.5
- removed net N$16: J2A.CAM1_DP0, J5.3
- removed net N$17: J2A.CAM1_DN0, J5.2
- removed net N$18: J2A.CAM0_DN0, J4.2
- removed net N$19: J2A.CAM0_DP0, J4.3
- removed net N$2: C1.1, J1B.GPIO0-27_VDD@1, J1B.GPIO0-27_VDD@2, R2.2, R3.2
- removed net N$20: J2A.CAM0_DN1, J4.5
- removed net N$21: J2A.CAM0_DP1, J4.6
- removed net N$22: J2A.CAM0_CN, J4.8
- removed net N$23: J2A.CAM0_CP, J4.9
- removed net N$24: J2A.HDMI_D2_P, U3.D2+
- removed net N$25: J2A.HDMI_D2_N, U3.D2-
- removed net N$26: J2A.HDMI_D1_N, U3.D1-
- removed net N$27: J2A.HDMI_D1_P, U3.D1+
- removed net N$28: J2A.HDMI_D0_P, U3.D0+
- removed net N$29: J2A.HDMI_D0_N, U3.D0-
- removed net N$3: J2A.GPIO11, J3.GPIO11
- removed net N$30: J2B.HDMI_HPD_N_1V8, R55.1
- removed net N$31: Q2.S, Q3.D, R44.1
- removed net N$32: DQ6.C, R44.2
- removed net N$33: Q2.G, Q4.C, R1.2
- removed net N$34: DQ1.C, R12.2
- removed net N$35: DQ2.C, R25.2
- removed net N$36: L2.1, U2.SW2
- removed net N$37: R11.2, R14.2, U2.FB2
- removed net N$38: R9.2, U2.PGND_2
- removed net N$39: L3.1, U2.SW1
- removed net N$4: C2.1, J1B.GPIO28-45_VDD@1, J1B.GPIO28-45_VDD@2, R5.2, R6.2
- removed net N$40: R8.2, U2.PGND_4
- removed net N$41: S2A.B, X1.1
- removed net N$6: J2A.GPIO10, J3.GPIO10
- removed net N$7: J2A.GPIO9, J3.GPIO09
- removed net N$8: J2A.GPIO22, J3.GPIO22
- removed net N$9: J2A.GPIO27, J3.GPIO27
- removed net SD_DETECT: J2A.GPIO34
- net +1.8V: now also C29.1, C30.1, C31.1, C32.1; no longer C102.1, C103.1, C13.1, C15.1, J1B.1V8@1, J1B.1V8@2, J1B.1V8@3, J1B.1V8@4, R3.1, R4.2, R55.2, R6.1
- net +2.5V: now also C42.1, C43.1, C44.1, C46.1, C47.1, R1.2; no longer C10.1, C17.1, C31.1, C32.1, C8.1, R45.2
- net +3.3V: now also C10.1, C11.1, C13.1, C14.1, C15.1, C17.1, C18.1, C19.1, C20.1, C21.1, C22.1, C23.1, C24.1, C25.1, C28.1, C38.1, C39.1, C40.1, C41.1, R1.1; no longer C3.1, C30.1, C33.1, C4.1, C46.1, C5.1, C52.1, C58.1, C6.1, C69.1, C7.1, C70.1, C71.1, C72.1, C76.1, C77.1, C78.1, C79.1, C80.1, C81.1, C82.1, C83.1, C84.1, C85.1, C88.1, C91.1, DQ1.A, DQ6.A, J1B.3V3@1, J1B.3V3@2, J1B.3V3@3, J1B.3V3@4, J3.3V3@1, J3.3V3@2, J4.15, J5.15, L3.2, R16.1, R17.1, R2.1, R20.1, R21.1, R22.1, R45.1, R49.2, R5.1, R50.2
- net +5V: now also C1.1, C2.1, C3.1, C4.1, C49.1, C5.1, C6.1, C7.1, C8.1, D1.A, D1.C, R3.2; no longer C11.1, C23.1, C24.1, C34.1, C36.1, C37.1, C38.1, C39.1, C40.1, C41.1, C47.1, DQ2.A, F1.1, F1.2, J3.5V0@1, J3.5V0@2, Q4.E, R15.1, R7.2, R8.1, R9.1, S2A.COMMON, U2.EN1, U2.EN2, VD4.A, VD4.C
- net GND: now also C14.2, C20.2, C42.2, C43.2, C44.2, C49.2, C50.2; no longer C102.2, C103.2, C52.2, C58.2, C69.2, C70.2, C71.2, C72.2, C76.2, C77.2, C78.2, C79.2, C80.2, C81.2, C82.2, C83.2, C84.2, C85.2, C88.2, C91.2, J1C.GND@1, J1C.GND@10, J1C.GND@11, J1C.GND@12, J1C.GND@13, J1C.GND@14, J1C.GND@15, J1C.GND@16, J1C.GND@17, J1C.GND@18, J1C.GND@19, J1C.GND@2, J1C.GND@20, J1C.GND@21, J1C.GND@22, J1C.GND@23, J1C.GND@24, J1C.GND@25, J1C.GND@26, J1C.GND@27, J1C.GND@28, J1C.GND@29, J1C.GND@3, J1C.GND@30, J1C.GND@31, J1C.GND@32, J1C.GND@33, J1C.GND@34, J1C.GND@35, J1C.GND@36, J1C.GND@37, J1C.GND@38, J1C.GND@39, J1C.GND@4, J1C.GND@40, J1C.GND@41, J1C.GND@42, J1C.GND@43, J1C.GND@44, J1C.GND@45, J1C.GND@46, J1C.GND@47, J1C.GND@48, J1C.GND@49, J1C.GND@5, J1C.GND@50, J1C.GND@51, J1C.GND@52, J1C.GND@53, J1C.GND@54, J1C.GND@55, J1C.GND@56, J1C.GND@57, J1C.GND@58, J1C.GND@59, J1C.GND@6, J1C.GND@60, J1C.GND@61, J1C.GND@7, J1C.GND@8, J1C.GND@9, J3.GND@1, J3.GND@5, J3.GND@6, J3.GND@8, J4.1, J4.10, J4.4, J4.7, J5.1, J5.10, J5.4, J5.7, Q3.S, R1.1, R12.1, R13.1, R14.1, R23.1, R24.1, R25.1, U2.AGND, U2.EPAD, U2.GND, U2.GND_2, U2.PGND, U2.PGND1, U2.PGND1_2, U2.PGND_3, X1.2
- net N$5: now also C50.1, R3.1; no longer C25.1, R7.1
- net VBATT: now also C33.1, C34.1, C36.1, C37.1; no longer C18.1, C19.1, C21.1, C22.1, J1B.VBAT@1, J1B.VBAT@2, J1B.VBAT@3, J1B.VBAT@4, R15.2, R17.2
