File: distributed-vision/DistributedVisionSchematicPage1_3.brd (EAGLE design)
At the start: 218 x 149 mm, 216 parts, among them IC1 IPB180N06S4-H1, J10 USBR-A-D-F-O-TH, J12 ARJM11C7-104-AB-EW2, J2 RASPBERRRY_COMPUTE_CM3, J3 XS10, J5 1981584-1, J6 DM3D-SF, J7 10029449-111RLF, J8 1-84952-5, J9 1-84952-5, Q1 AP2331SA-7, Q2 BSS127, Q3 BSS127, Q4 BSS127, Q5 PSMN014-40YS, Q6 25 MHz, U11 IFX91041, U12 TPS26600PWPR, U2 LM26420XMH, U3 LAN9513-JZXQFN64_9X9MC_MCH-M, U4 ESD224, U5 FSUSB42MUX, U6 SP3003-02, U7 SP3003-02, U8 SP3003-02, U9 SP3003-02, X1 JST-XH-02-PIN-LONG-PAD

Commit message: Board/Schematic Update
Parts:
- removed C54, C59: 100n, rcl:C0402
- removed C55, C67: 10n, rcl:C0402
- removed C56: 1nF, rcl:C0402
- removed C57: 10u, rcl:C0402
- removed D1, D2: GREEN, RoboJackets-LEDs:LED-0603
- removed IC1: IPB180N06S4-H1, infineon:PG-TO263-7-3
- removed J5: 1981584-1, RoboJackets-Connectors:TE_1981584-1
- removed JP2: (no value), RoboJackets-Connectors:1X04
- removed L3, L6: 2A 120r, RoboJackets-Inductors:0805
- removed LED1, LED2, LED3: LAP4-BOTTOM, led:P47F-BOTTOM
- removed R12, R25: 470r, rcl:R0603
- removed R18: 47k, RoboJackets-Resistors:RC0805N
- removed R19, R51: 4k7, RoboJackets-Resistors:RC0805N
- removed R29: 470r, RoboJackets-Resistors:RC0805N
- removed R41: 1M, RoboJackets-Resistors:RC0805N
- removed T1: (no value), transistor:SC59-BEC
- removed U5: FSUSB42MUX, distributed-vision:10-MSOP
- removed U6, U7: SP3003-02, distributed-vision:SC70-5
- R16, R20, R49, R50: value 4k7 -> 4.7k
- moved S2 213.6 mm to (96.7, 78.7)
- moved Q5 211.2 mm to (77.6, 182.7)
- moved H2 175.6 mm to (27.5, -41.7)
- moved L9 162.5 mm to (10.9, 8.80)
- moved U3 151.2 mm to (10.4, 48.4)
- moved F2 135.8 mm to (71.0, 87.4)
- moved U2 122.4 mm to (9.59, 64.7), turned to 90 degrees
- moved J7 111.1 mm to (210.7, 71.7), turned to 90 degrees
- moved J12 103.0 mm to (12.2, -28.8)
- moved U11 74.6 mm to (8.93, 76.4)
- moved J10 64.0 mm to (77.2, -39.8)
- moved U12 41.2 mm to (7.87, 93.4)
- moved J9 35.0 mm to (206.4, 9.25)
Connections:
- removed net D+: U5.3
- removed net D-: U5.4
- removed net IO1: J5.3, U5.7, U6.6
- removed net IO2: J5.2, U5.6, U6.4
- removed net N$57: R29.2, U3.20
- removed net N$60: LED3.C, R29.1
- removed net N$68: IC1.8, R18.1, U5.2
- removed net N$72: J5.1, L3.2, U6.3
- removed net N$73: C57.1, C59.1, C67.1, JP2.1, L6.2, U7.3
- removed net N$75: C54.1, C55.1, R18.2
- removed net VDD33A_2: U3.5
- removed net VDD33A_3: U3.10
- removed net VDD33IO_2: U3.19
- removed net VDD33IO_3: U3.27
- new net +3.3V: C12.1, C4.1, C5.1, C7.1, U3.10, U3.19, U3.27, U3.5
- new net N$1: J3.6
- net +5V: no longer D2.A
- net FB1: no longer C12.1, C4.1, C5.1, C7.1, D1.A
- net GND: no longer C54.2, C55.2, C56.1, C56.2, C57.2, C59.2, C67.2, IC1.2, IC1.3, IC1.5, IC1.6, IC1.7, J3.6, J5.10, J5.11, J5.5, J5.6, J5.7, J5.8, J5.9, JP2.4, R12.1, R19.2, R25.1, R41.1, R41.2, R51.1, R51.2, T1.E, U5.10, U5.5, U6.2, U7.2
- net N$61: no longer T1.C
- net NLINKA_LED: no longer J12.L2, LED2.C
- net NSPD_LED: no longer J12.L4, LED1.C
- net TX_N: no longer D2.C, R25.2
- net TX_P: no longer D1.C, R12.2
- net USBDM0: no longer U5.8
- net USBDM4: no longer JP2.2, U3.6, U7.4, U7.6
- net USBDP0: no longer U5.9
- net USBDP4: no longer JP2.3, U3.7
- net VCC: no longer IC1.1, L3.1, L6.1, LED1.A, LED2.A, LED3.A, R19.1, U5.1
