File: distributed-vision/DistributedVisionSchematicPagePRAC.sch (EAGLE design)
At the start: 157 parts, among them J1 USBR-A-D-F-O-TH, J12 ARJM11C7-104-AB-EW2, J2 RASPBERRRY_COMPUTE_CM3, J6 DM3D-SF, J8 1-84952-5, J9 1-84952-5, Q2 BSS127, Q3 BSS127, Q7 25 MHz, U1 LM26420XMH, U11 IFX91041, U12 TPS26600PWPR, U3 LAN9513-JZXQFN64_9X9MC_MCH-M, U8 SP3003-02, U9 SP3003-02, X1 JST-XH-02-PIN-LONG-PAD

Commit message: Version 2 of April Tag Board with Design Review Changes
Parts:
- removed J1: USBR-A-D-F-O-TH, USBR-A-D-F-O-TH:USBR-A-D-F-O-TH
- removed Q7: 25 MHz, crystal:FA-20H
- removed R2: (no value), rcl:R-US_R0603
- added C11, C3, C34, C49: (no value), rcl:C-USC0603
- added C130, C131: 18pF, rcl:C-USC0603
- added C132: 22uF, SparkFun-Capacitors:22UF-POLAR-PANASONIC_C-35V-20%
- added C133, C134, C135, C136, C137, C138, C142, C148: 0.1uF, adafruit:C-USC0402
- added C139: 10000pF, adafruit:C-USC0402
- added C140: 4.7uF, rcl:C-USC0603
- added C141: 22uF, rcl:C-USC0603
- added C144, C145: 0.1uF, adafruit:C-USC0603
- added C146, C147: 1uF, rcl:C-USC0603
- added C36, C39, C40, C48, C96: 100n, rcl:C-USC0603
- added C37: 22u, rcl:C-USC0603
- added C38, C41: 10n, rcl:C-USC0603
- added C47: 10u, rcl:C-USC0603
- added C54, C59: 100n, rcl:C-USC0402
- added C55, C67: 10n, rcl:C-USC0402
- added C56: 1nF, rcl:C-USC0402
- added C57: 10u, rcl:C-USC0402
- added D1, D2: GREEN, RoboJackets-LEDs:LED-GREEN0603
- added D11: NTS260ESFT3G, ethernet_poe:NTS260ESFT3G
- added D4: 60V, RoboJackets-Diodes:DFLS160-7
- added D8: YLW, led:LEDCHIP-LED0603
- added D9: BLU, led:LEDCHIP-LED0603
- added FB1: 742792023, ethernet_poe:742792023
- added IC1: IPB180N06S4-H1, infineon:IPB180N06S4-H1
- added J10: USBR-A-D-F-O-TH, distributed-vision:USBR-A-D-F-O-TH
- added J11: (no value), SparkFun-Connectors:CONN_07
- added J3: XS10, distributed-vision:XS10
- added J4: (no value), SparkFun-Connectors:CONN_05
- added J5: 1981584-1, RoboJackets-Connectors:1981584-1
- added J7: 10029449-111RLF, distributed-vision:10029449-111RLF
- added JP2: (no value), RoboJackets-Connectors:PINHD-1X4
- added L3, L6: 2A 120r, RoboJackets-Inductors:INDUCTOR_0805
- added L5: MPZ2012S601AT000, POE:MPZ2012S601AT000
- added LED1, LED2, LED3: LAP4-BOTTOM, led:LAP4-BOTTOM
- added Q1: AP2331SA-7, distributed-vision:AP2331SA-7
- added Q4: BSS127, RoboJackets-Discrete:BSS127
- added Q5: PSMN014-40YS, RoboJackets-Discrete:PSMN014-40YS
- added Q6: 25 MHz, crystal:FA-20H
- added R100, R99: 470, rcl:R-US_R0603
- added R12, R25: 470r, rcl:R-US_R0603
- added R18, R56: 47k, RoboJackets-Resistors:ERJ-L06KF50MV
- added R19, R51: 4k7, RoboJackets-Resistors:ERJ-L06KF50MV
- added R29: 470r, RoboJackets-Resistors:ERJ-L06KF50MV
- added R38, R42, R43, R46, R47, R48: (no value), rcl:R-US_R0603
- added R41: 1M, RoboJackets-Resistors:ERJ-L06KF50MV
- added R49, R50, R52, R53, R54: 4k7, rcl:R-US_R0603
- added R55: 47k, rcl:R-US_R0603
- added R88, R89, R90, R91, R92, R95: 10k, rcl:R-US_R0603
- added R93: 1M, adafruit:R-US_R0402
- added R94: 12.4k, 1%, rcl:R-US_R0603
- added S1: KMR2, RoboJackets-Switches:KMR2
- added T1: (no value), transistor:MUN2211T1-NPN_DRIVER-SC59-BEC
- added U10: AZ1117EH-3.3TRG1, ethernet_poe:AZ1117EH-3.3TRG1
- added U2: LM26420XMH, distributed-vision:LM26420XMH
- added U4: ESD224, distributed-vision:ESD224
- added U5: FSUSB42MUX, distributed-vision:FSUSB42MUX
- added U6, U7: SP3003-02, distributed-vision:SP3003-02
- added X2: 25MHz, ethernet_poe_v2.1:ABM10W-25.0000MHZ-6-K1Z-T3
- C20, C51, C75, C86: value 10n -> (none)
- C23, C24: value 22u -> (none)
- C25: value 470n -> (none)
- C42, C50, C83: value 100n -> (none)
- C43, C44: value 4u7 -> (none)
- F1: value 2A -> (none)
- L1, L2: value 4A -> 1uH
- R10: value 31.6k -> 31k6
- R11: value 12.7k -> 12k7
- R13: value 10k -> (none)
- R16, R20, R21, R22, R28, R31: value 4.7k -> 4k7
- R27: value 12.4k -> 12k4
- R30, R32: value 4.7k -> 470r
- R7: value 5r1 -> (none)
- RN42, RN43: value 22 -> (none)
- U1: value LM26420XMH -> W5500; device LM26420XMH:LM26420XMH -> ethernet_poe:W5500
Connections:
- removed net +3.3V: C10.1, C12.1, C17.1, C20.1, C26.1, C27.1, C4.1, C42.1, C43.1, C44.1, C45.1, C46.1, C5.1, C50.1, C51.1, C52.1, C58.1, C69.1, C7.1, C70.1, C71.1, C72.1, C75.1, C76.1, C77.1, C8.1, C86.1, C9.1, D6.A, J2B.3V3@1, J2B.3V3@2, J2B.3V3@3, J2B.3V3@4, J2B.GPIO0-27_VDD@2, J2B.GPIO28-45_VDD@2, J2B.VDAC@1, J2B.VDAC@2, J2D.SDX_VDD, J2D.SDX_VDD1, J6.4, J8.15, J9.15, L8.1, R10.2, R16.1, R20.1, R21.1, R22.1, R28.PIN2, R31.PIN2, R40.PIN2, R74.1, R75.1, R98.1, U3.TEST3, U3.VBUS_DET, U3.VDD33A, U3.VDD33A_2, U3.VDD33A_3, U3.VDD33A_4, U3.VDD33A_5, U3.VDD33A_6, U3.VDD33A_7, U3.VDD33IO, U3.VDD33IO_2, U3.VDD33IO_3, U3.VDD33IO_4, U3.VDD33IO_5
- removed net +3.3V-A: C16.1, C33.1, C6.1, C78.1, C79.1, C80.1, C81.1, C82.1, C83.1, C84.1, C85.1, C88.1, C91.1, L8.2
- removed net BD+: J1.D1+, U9.IO2
- removed net BVCC: J1.VCC1, S2A.B, X1.1
- removed net TVCC: C68.1, C73.1, J1.VCC2, L7.2, U8.VCC, U9.VCC
- removed net USBDM3: U3.USBDM3
- removed net USBDM4: L2.1, U1.SW2
- removed net USBDP3: J1.D2+, J1.D2-, U3.USBDP3, U8.IO1, U8.IO2
- removed net USBDP4: R14.2, U1.FB2
- removed net USB_DM: U3.USBDM0
- removed net USB_DP: U3.USBDP0
- removed net USB_OTGID: J2A.USB_OTGID, R2.2
- removed net VDD18CORE: C14.1, C60.1, C61.1, C62.1, R13.2, U1.FB1, U3.VDD18CORE, U3.VDD18CORE_2
- new net !INT: J11.1, R89.2, U1.!INTN
- new net !RST: C148.1, J4.2, R95.1, S1.2, U1.!RSTN
- new net !SCS: J11.5, R88.2, U1.!SCSN
- new net +2.5V: C10.1, C17.1, C8.1
- new net +3V3_D: C141.1, C142.1, C145.1, C147.1, D11.2, FB1.2, J4.4, R100.1, R74.1, R75.1, R88.1, R89.1, R90.2, R91.2, R92.2, R95.2, R98.1, R99.1, U1.VDD, U10.OUT
- new net 3V3: C3.1, J3.3V3@1, J3.3V3@2
- new net 3V3_LED1: D8.A, R99.2
- new net 3V3_LED2: D9.A, R100.2
- new net 5V/R53: J2A.HDMI_SDA, J7.16, R53.1, U4.IO4_C
- new net 5V/R54: J7.15
- new net ACTLED: D8.C, U1.ACTLED
- new net DUPLED: D9.C, U1.DUPLED
- new net FB2: C28.1, C29.1, L2.2, R11.1
- new net GPIO02: J2A.GPIO2, J3.GPIO02, R49.1
- new net GPIO03: J2A.GPIO3, J3.GPIO03, R50.1
- new net GPIO04: J2A.GPIO4, J3.GPIO04
- new net GPIO05: J2A.GPIO5, J3.GPIO05
- new net GPIO06: J2A.GPIO6, J3.GPIO06
- new net GPIO07: J2A.GPIO7, J3.GPIO07
- new net GPIO08: J2A.GPIO8, J3.GPIO08
- new net GPIO09: J2A.GPIO9, J3.GPIO09
- new net GPIO10: J2A.GPIO10, J3.GPIO10
- new net GPIO11: J2A.GPIO11, J3.GPIO11
- new net GPIO12: J2A.GPIO12, J3.GPIO12
- new net GPIO13: J2A.GPIO13, J3.GPIO13
- new net GPIO14: J2A.GPIO14, J3.GPIO14
- new net GPIO15: J2A.GPIO15, J3.GPIO15
- new net GPIO16: J2A.GPIO16, J3.GPIO16
- new net GPIO17: J2A.GPIO17, J3.GPIO17
- new net GPIO18: J2A.GPIO18, J3.GPIO18
- new net GPIO19: J2A.GPIO19, J3.GPIO19
- new net GPIO20: J2A.GPIO20, J3.GPIO20
- new net GPIO21: J2A.GPIO21, J3.GPIO21
- new net GPIO22: J2A.GPIO22
- new net GPIO23: J2A.GPIO23, J3.GPIO23
- new net GPIO24: J2A.GPIO24, J3.GPIO24
- new net GPIO25: J2A.GPIO25, J3.GPIO25
- new net GPIO26: J2A.GPIO26, J3.GPIO26
- new net GPIO27: J2A.GPIO27, J3.GPIO27
- new net HDMI_CLK_N: J2A.HDMI_CLK_N, J7.12
- new net HDMI_CLK_P: J2A.HDMI_CLK_P, J7.10
- new net HDMI_D0_N: J2A.HDMI_D0_N, J7.9
- new net HDMI_D0_P: J2A.HDMI_D0_P, J7.7
- new net HDMI_D1_N: J2A.HDMI_D1_N, J7.6
- new net HDMI_D1_P: J2A.HDMI_D1_P, J7.4
- new net HDMI_D2_N: J2A.HDMI_D2_N, J7.3
- new net HDMI_D2_P: J2A.HDMI_D2_P, J7.1
- new net HDMI_SCL: J2A.HDMI_SCL, R54.1, U4.IO3_C
- new net MISO: J11.3, U1.MISO
- new net MOSI: J11.2, U1.MOSI
- new net N$11: C131.1, R93.1, U1.XO, X2.OUT
- new net N$12: C75.1, J2B.GPIO0-27_VDD@1, J2B.GPIO0-27_VDD@2, R38.2, R42.2
- new net N$13: C130.1, R93.2, U1.XI, X2.IN
- new net N$17: U5.D+
- new net N$17/1.6C: J2A.USB_DP
- new net N$18: U5.D-
- new net N$18/1.6B: J2A.USB_DM
- new net N$19: R51.PIN1
- new net N$2: C139.1, U1.1V2O
- new net N$21: R94.2, U1.EXRES1
- new net N$22: U3.USBDP0, U5.HSD2+
- new net N$23: U3.USBDM0, U5.HSD2-
- new net N$24: C86.1, J2B.GPIO28-45_VDD@1, J2B.GPIO28-45_VDD@2, R43.2, R46.2
- new net N$26: J5.3, U5.HSD1+, U6.IO1
- new net N$27: J5.2, U5.HSD1-, U6.IO2
- new net N$3: C140.1, U1.TOCAP
- new net N$30: J10.BD+, J2B.HDMI_HPD_N_1V8, Q5.S, R55.1, U9.IO2
- new net N$36: JP2.2, L2.1, U2.SW2, U3.USBDM4, U7.IO1, U7.IO2
- new net N$37: JP2.3, R11.2, R14.2, U2.FB2, U3.USBDP4
- new net N$41: J10.BVCC, S2A.B, X1.1
- new net N$42: C68.1, C73.1, J10.TVCC, L7.2, U8.VCC, U9.VCC
- new net N$45: J7.19, Q5.G, R56.PIN2
- new net N$52: J2A.HDMI_CEC, Q4.D, R52.1
- new net N$53: Q4.S, U4.IO2_C
- new net N$57: R29.PIN2, U3.NFDX_LED/GPIO0
- new net N$60: LED3.C, R29.PIN1
- new net N$68: IC1.D, R18.PIN1, U5.SEL
- new net N$7: R90.1, U1.PMODE0
- new net N$72: J5.1, L3.2, U6.VCC
- new net N$73: C57.1, C59.1, C67.1, JP2.1, L6.2, U7.VCC
- new net N$75: C54.1, C55.1, R18.PIN2
- new net N$8: R91.1, U1.PMODE1
- new net N$9: R92.1, U1.PMODE2
- new net NS$19/1.6B: J2A.USB_OTGID
- new net SCLK: J11.4, U1.SCLK
- new net SD_DETECT: J2A.GPIO34
- new net VCC: IC1.G, L3.1, L6.1, L7.1, LED1.A, LED2.A, LED3.A, R19.PIN1, R28.PIN2, R31.PIN2, R40.PIN2, U3.TEST3, U3.VBUS_DET, U3.VDD33A, U3.VDD33IO, U5.VCC
- net +1.8V: now also R38.1, R43.1, R55.2; no longer C28.1, C29.1, L2.2, R11.2
- net +24V_FUSE: now also J4.1
- net +3V3_A: now also C132.+, C133.1, C134.1, C135.1, C136.1, C137.1, C138.1, C144.1, FB1.1, U1.AVDD
- net +5V: now also C11.1, C146.1, C34.1, C36.1, C37.1, C38.1, C39.1, C40.1, C41.1, C47.1, C48.1, C96.1, D11.1, D2.A, D4.A, D4.C, J3.5V0@1, J3.5V0@2, J4.3, J7.18, Q1.IN, Q1.OUT, Q4.G, R47.1, R53.2, R54.2, U10.IN, U2.EN1, U2.EN2, U2.VIND1, U2.VIND1_2, U2.VIND2, U2.VIND2_2, U4.IO1_C, U4.IO1_S, U4.IO3_S, U4.IO4_S; no longer L7.1, U1.EN1, U1.EN2, U1.VIND1, U1.VIND2
- net 24_LOAD: now also J11.7
- net AGND: now also J12.CHASSIS1, J12.CHASSIS2, L5.2
- net FB1: now also C12.1, C16.1, C20.1, C26.1, C27.1, C33.1, C4.1, C42.1, C43.1, C44.1, C45.1, C46.1, C49.1, C5.1, C50.1, C51.1, C52.1, C58.1, C6.1, C69.1, C7.1, C70.1, C71.1, C72.1, C76.1, C77.1, C78.1, C79.1, C80.1, C81.1, C82.1, C83.1, C84.1, C85.1, C88.1, C9.1, C91.1, D1.A, D6.A, J2B.3V3@1, J2B.3V3@2, J2B.3V3@3, J2B.3V3@4, J2D.SDX_VDD, J2D.SDX_VDD1, J6.4, J8.15, J9.15, L8.1, L8.2, R16.1, R20.1, R21.1, R22.1, R42.1, R46.1, R48.1, R49.2, R50.2, R52.2
- net GND: now also C11.2, C130.2, C131.2, C132.-, C133.2, C134.2, C135.2, C136.2, C137.2, C138.2, C139.2, C140.2, C141.2, C142.2, C144.2, C145.2, C146.2, C147.2, C148.2, C3.2, C34.2, C36.2, C37.2, C38.2, C39.2, C40.2, C41.2, C47.2, C48.2, C49.2, C54.2, C55.2, C56.1, C56.2, C57.2, C59.2, C67.2, C96.2, IC1.S, J10.BGND, J10.TGND, J11.6, J3.GND@1, J3.GND@5, J3.GND@6, J3.GND@7, J3.GND@8, J4.5, J5.5, J5.SHIELD, J7.11, J7.17, J7.2, J7.5, J7.8, JP2.4, L5.1, Q1.GND, Q5.D, R12.1, R19.PIN2, R25.1, R41.PIN1, R41.PIN2, R51.PIN2, R56.PIN1, R94.1, S1.1, T1.E, U10.ADJ/GND, U2.AGND, U2.EPAD, U2.GND, U2.GND_2, U2.PGND, U2.PGND1, U2.PGND1_2, U2.PGND_3, U4.GND@1, U4.GND@2, U5.!OE, U5.GND, U6.GND, U7.GND, X2.SHD1, X2.SHD2; no longer J1.GND1, J1.GND2, J12.CHASSIS1, J12.CHASSIS2, R2.1, U1.EPAD, U1.PGND, U1.PGND1, U1.PGND_3, U3.EPAD
- net N$1: now also C14.1, C60.1, C61.1, C62.1, R10.2, R13.2, U2.FB1, U3.VDD18CORE; no longer R11.1
- net N$31: now also J10.TD-, U3.USBDM3, U8.IO1, U8.IO2
- net N$32: now also J10.TD+, U3.USBDP3
- net N$40: now also U2.PGND_4; no longer U1.PGND_4
- net N$5: now also U2.VINC; no longer U1.VINC
- net N$61: now also T1.C
- net N$64: now also Q6.2; no longer Q7.3
- net N$65: now also Q6.4; no longer Q7.1
- net N$66: now also Q6.1; no longer Q7.4
- net N$67: now also Q6.3; no longer Q7.2
- net NLINKA_LED: now also J12.G_LED-, LED2.C, U1.LINKLED
- net NSPD_LED: now also J12.Y_LED-, LED1.C, U1.SPDLED
- net RX_N: now also U1.RXN, U2.SW1; no longer U1.SW1
- net RX_P: now also U1.RXP, U2.PGND_2; no longer U1.PGND_2
- net TX_N: now also D2.C, R25.2, U1.TXN
- net TX_P: now also D1.C, R12.2, U1.TXP
- net USBDM2: now also J10.BD-; no longer J1.D1-
- net VBATT: now also R47.2, R48.2
Other:
- note added: "1A Rated"
- note added: "3.3V Analog"
- note added: "5V FROM USB BOOT"
- note added: "5V to 3.3V"
- note added: "Chassis Ground"
- note added: "Control"
- note added: "Filtering"
- note added: "HDMI"
- note added: "HDMI POWER"
- note added: "Headers"
- note added: "NOTE: This pi filter isolates the digital and analog 3.3V power supplies by attenuating differential mode noise."
- note added: "Power (5V-3.3V)"
- note added: "RASPBERRY PI HEADER"
- note added: "RC to debounce switch"
- note added: "Reset"
- note removed: "NO CONNECT"
- moved on the sheet: C127, C128, C129, C20, C42, C43, C44, C50, C51, C75, C86, D3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
